File: pcb/power/power.kicad_sch (KiCad schematic)
At the start: 0 parts

Commit message: hardware: update DRV8874 power schematic and PCB project
Parts:
- added C1, C102, C92: 100 nF 25 V, Capacitor_SMD:C_0603_1608Metric, symbol EdgePower:C
- added C10, C11, C30, C31: 10u/50V, Capacitor_SMD:C_1210_3225Metric, symbol EdgePower:C
- added C100, C90: 22 nF 25 V, Capacitor_SMD:C_0603_1608Metric, symbol EdgePower:C
- added C101, C91: 100 nF 16 V, Capacitor_SMD:C_0603_1608Metric, symbol EdgePower:C
- added C103, C93: 47 uF 25 V, Capacitor_SMD:C_1210_3225Metric, symbol EdgePower:C
- added C12, C13, C14: 47u/10V, Capacitor_SMD:C_1210_3225Metric, symbol EdgePower:C
- added C2, C4: 470 uF 25 V, Capacitor_THT:CP_Radial_D10.0mm_P5.00mm, symbol EdgePower:C
- added C3: 10 nF, Capacitor_SMD:C_0603_1608Metric, symbol EdgePower:C
- added C32, C33, C34: 47u/25V, Capacitor_SMD:C_1210_3225Metric, symbol EdgePower:C
- added C50: 4.7 uF 10V, Capacitor_SMD:C_0805_2012Metric, symbol EdgePower:C
- added C51, C52: 22 uF 10V, Capacitor_SMD:C_0805_2012Metric, symbol EdgePower:C
- added C80: 150 uF 10V, Capacitor_THT:CP_Radial_D8.0mm_P3.50mm, symbol EdgePower:C
- added C81: 100 nF 10V, Capacitor_SMD:C_0603_1608Metric, symbol EdgePower:C
- added C82: 10 uF 10V, Capacitor_SMD:C_0805_2012Metric, symbol EdgePower:C
- added D1: SMBJ15A, Diode_SMD:D_SMB, symbol EdgePower:TVS
- added D2: SMBJ15A 待核, Diode_SMD:D_SMB, symbol EdgePower:TVS
- added F1: 15 A 待核, symbol EdgePower:Fuse
- added F2, F5, F8: 4 A 待核, symbol EdgePower:Fuse
- added F3: 3.5 A 待核, symbol EdgePower:Fuse
- added F4: 10 A 待核, symbol EdgePower:Fuse
- added F6, F7: 3 A 待核, symbol EdgePower:Fuse
- added J1: XT60 母座, Connector_AMASS:AMASS_XT60PW-F_1x02_P7.20mm_Horizontal, symbol EdgePower:XT60_F
- added J11: 步进驱动 1 供电, symbol EdgePower:Conn_2
- added J12: 步进驱动 2 供电, symbol EdgePower:Conn_2
- added J13: L 驱动控制, symbol EdgePower:DRV_CTRL
- added J14: R 驱动控制, symbol EdgePower:DRV_CTRL
- added J15: L MG513 电机, symbol EdgePower:Conn_2
- added J16: R MG513 电机, symbol EdgePower:Conn_2
- added J2: 电池总压检测, symbol EdgePower:Conn_2
- added J3: USB-C 5V 输出, Connector_USB:USB_C_Receptacle_GCT_USB4125-xx-x_6P_TopMnt_Horizontal, symbol EdgePower:USB_C_Source_6P
- added J4: ACG720 9V 输入, symbol EdgePower:Conn_2
- added J5: ICM-42688-P 供电, symbol EdgePower:Conn_2
- added J6: VL53L1X 供电, symbol EdgePower:Conn_2
- added J7: 左编码器供电, symbol EdgePower:Conn_2
- added J8: 右编码器供电, symbol EdgePower:Conn_2
- added J9: 常闭急停回路, symbol EdgePower:Conn_2_Right
- added L1: 2.2 uH Isat>=3A, symbol EdgePower:Inductor
- added Q1: CSD18540Q5B, symbol EdgePower:N_FET_ideal_diode
- added R1: 180 k 1%, Resistor_SMD:R_0603_1608Metric, symbol EdgePower:R
- added R11: 40.2 k 1%, Resistor_SMD:R_0603_1608Metric, symbol EdgePower:R
- added R12, R32, R83, R93: 10 k 1%, Resistor_SMD:R_0603_1608Metric, symbol EdgePower:R
- added R13: 13 k, Resistor_SMD:R_0603_1608Metric, symbol EdgePower:R
- added R2: 47 k 1%, Resistor_SMD:R_0603_1608Metric, symbol EdgePower:R
- added R24, R51: 100 k 1%, Resistor_SMD:R_0603_1608Metric, symbol EdgePower:R
- added R31: 80.6 k 1%, Resistor_SMD:R_0603_1608Metric, symbol EdgePower:R
- added R33: 6.34 k, Resistor_SMD:R_0603_1608Metric, symbol EdgePower:R
- added R50: 453 k 1%, Resistor_SMD:R_0603_1608Metric, symbol EdgePower:R
- added R80, R90: 13 k 1%, Resistor_SMD:R_0603_1608Metric, symbol EdgePower:R
- added R81, R91: 20 k 1%, Resistor_SMD:R_0603_1608Metric, symbol EdgePower:R
- added R82, R92: 1.8 k 1%, Resistor_SMD:R_0603_1608Metric, symbol EdgePower:R
- added SW1: 总开关≥20A DC, symbol EdgePower:Switch
- added U1: LM74700QDBVRQ1, Package_TO_SOT_SMD:SOT-23-6, symbol EdgePower:LM74700_Q1
- added U2, U3: TPSM63606RDLR, symbol EdgePower:TPSM63606
- added U4: TLV62569DBVR, Package_TO_SOT_SMD:SOT-23-5, symbol EdgePower:TLV62569DBV
- added U6: TPS25810RVCT, symbol EdgePower:TPS25810RVC
- added U7, U8: DRV8874PWP, symbol EdgePower:DRV8874PWP
Connections:
- new net: R80.2, R81.1, U7.5 (VREF)
- new net: F7.2, J12.1 (+)
- new net: J13.4 (nFAULT), R83.2, U7.4 (nFAULT)
- new net: C80.1, C81.1, F2.2, U6.2 (IN1), U6.3 (IN1), U6.4 (IN2), U6.5 (AUX), U6.6 (EN), U6.7 (CHG), U6.8 (CHG_HI)
- new net: C101.1, C102.1, C103.1, F8.2, U8.11 (VM)
- new net: J13.1 (PWM), U7.1 (EN/PWM)
- new net: J15.2 (-), U7.10 (OUT2)
- new net: C91.1, C92.1, C93.1, F5.2, U7.11 (VM)
- new net: C91.2, U7.12 (VCP)
- new net: C90.2, U7.13 (CPH)
- new net: C90.1, U7.14 (CPL)
- new net: J13.2 (DIR), U7.2 (PH/DIR)
- new net: J13.3 (nSLEEP), U7.3 (nSLEEP)
- new net: J13.5 (ISENSE), R82.1, U7.6 (IPROPI)
- new net: J15.1 (+), U7.8 (OUT1)
- new net: R50.2, R51.1, U4.5 (FB)
- new net: F3.2, J4.1 (+)
- new net: C3.1, J2.1 (+), R1.2, R2.1
- new net: R33.1, U3.12 (RT)
- new net: J16.1 (+), U8.8 (OUT1)
- new net: J16.2 (-), U8.10 (OUT2)
- new net: C1.1, U1.1 (VCAP)
- new net: C1.2, Q1.1 (S), SW1.2, U1.3 (EN), U1.6 (ANODE)
- new net: Q1.3 (G), U1.5 (GATE)
- new net: R31.2, R32.1, U3.10 (FB)
- new net: U3.3 (CBOOT), U3.4 (RBOOT)
- new net: J3.A5 (CC1), U6.11 (CC1)
- new net: J3.B5 (CC2), U6.13 (CC2)
- new net: J14.1 (PWM), U8.1 (EN/PWM)
- new net: J14.2 (DIR), U8.2 (PH/DIR)
- new net: J14.3 (nSLEEP), U8.3 (nSLEEP)
- new net: J14.4 (nFAULT), R93.2, U8.4 (nFAULT)
- new net: J14.5 (ISENSE), R92.1, U8.6 (IPROPI)
- new net: R90.2, R91.1, U8.5 (VREF)
- new net: F4.2, J9.1 (急停出)
- new net: R13.1, U2.12 (RT)
- new net: C101.2, U8.12 (VCP)
- new net: C100.2, U8.13 (CPH)
- new net: C100.1, U8.14 (CPL)
- new net: L1.1, U4.3 (SW)
- new net: R11.2, R12.1, U2.10 (FB)
- new net: R24.1, U6.10 (REF)
- new net: R24.2, U6.9 (REF_RTN)
- new net: F6.2, J11.1 (+)
- new net: F1.2, SW1.1
- new net: U2.3 (CBOOT), U2.4 (RBOOT)
- new net 3V3: C51.1, C52.1, J5.1 (+), J6.1 (+), J7.1 (+), J8.1 (+), L1.2, R50.1, R80.1, R83.1, R90.1, R93.1
- new net 5V_MAIN: C12.1, C13.1, C14.1, C50.1, F2.1, R11.1, U2.5 (VLDOIN), U2.8 (VOUT1), U2.9 (VOUT2), U4.1 (EN), U4.4 (VIN)
- new net 5V_USB: C82.1, J3.A9 (VBUS), J3.B9 (VBUS), U6.14 (OUT), U6.15 (OUT)
- new net 9V_FPGA: C32.1, C33.1, C34.1, F3.1, R31.1, U3.5 (VLDOIN), U3.8 (VOUT1), U3.9 (VOUT2)
- new net BAT_RAW: F1.1, J1.2 (+)
- new net GND: C10.2, C102.2, C103.2, C11.2, C12.2, C13.2, C14.2, C2.2, C3.2, C30.2, C31.2, C32.2, C33.2, C34.2, C4.2, C50.2, C51.2, C52.2, C80.2, C81.2, C82.2, C92.2, C93.2, D1.2 (A), D2.2 (A), J1.1 (-), J11.2 (-), J12.2 (-), J13.6 (GND), J14.6 (GND), J2.2 (-), J3.A12 (GND), J3.B12 (GND), J3.SH (SHIELD), J4.2 (-), J5.2 (-), J6.2 (-), J7.2 (-), J8.2 (-), R12.2, R13.2, R2.2, R32.2, R33.2, R51.2, R81.2, R82.2, R91.2, R92.2, U1.2 (GND), U2.11 (AGND), U2.17 (PGND), U2.18 (PGND), U2.19 (PGND), U2.20 (PGND), U2.6 (AGND), U3.11 (AGND), U3.17 (PGND), U3.18 (PGND), U3.19 (PGND), U3.20 (PGND), U3.6 (AGND), U4.2 (GND), U6.12 (GND), U6.21 (EP), U7.15 (GND), U7.16 (PMODE), U7.17 (EP), U7.7 (IMODE), U7.9 (PGND), U8.15 (GND), U8.16 (PMODE), U8.17 (EP), U8.7 (IMODE), U8.9 (PGND)
- new net MOTOR_ON: C4.1, D2.1 (K), F5.1, F6.1, F7.1, F8.1, J9.2 (急停回)
- new net VBAT_PROT: C10.1, C11.1, C2.1, C30.1, C31.1, D1.1 (K), F4.1, Q1.2 (D), R1.1, U1.4 (CATHODE), U2.1 (VIN1), U2.14 (EN/SYNC), U2.16 (VIN2), U3.1 (VIN1), U3.14 (EN/SYNC), U3.16 (VIN2)
- no-connect marks 0 -> 14
Other:
- note added: "01 电池输入与保护"
- note added: "02 5 V / 4 A 预留｜Lichee Pi 4A USB-C 供电"
- note added: "03 9 V / 3 A 预留｜ACG720 与 OV5640"
- note added: "04 3.3 V / ≥0.5 A｜传感器、编码器与驱动逻辑"
- note added: "05 动力母线与急停"
- note added: "06 有刷电机｜DRV8874 × 2｜PH/EN 控制"
- note added: "07 两台步进驱动模块（外置）"
- note added: "9V 降压级在电池接近 9V 时会掉压；须实测 FPGA 峰值电流。"
- note added: "DRV8874 VM 直连 3S 动力母线（满电 12.6V）；每台斩波阈值约 2.4A，须实测起动与散热。"
- note added: "EdgeMind 机器人｜3S 锂电池电源控制板｜原理图工程草案"
- note added: "J13 左轮 FPGA 控制"
- note added: "J14 右轮 FPGA 控制"
- note added: "Lichee Pi 4A 由 USB-C 线供电；TPS25810 检测连接后开启 5V，宣告 3A 并限流。"
- note added: "仅为原理图，尚未完成 PCB；使用旧电池前须检查单节状态、极性及保险丝额定值。"
- note added: "依据：TI DRV8874、LM74700-Q1、TPSM63606、TLV62569 数据手册；参数为设计初选，尚未实测验证。"
- note added: "急停仅切断驱动 VM；FPGA 还应主动拉低两颗 DRV8874 的 nSLEEP，并停用步进驱动。"
- note added: "投板前：实测 3S 电池状态、急停与回生瞬态、各路电流/温升、封装焊盘及输出极性。"
- note added: "此处四个接口只供电；传感器与编码器信号线另接 FPGA，不能默认耐受 5V。"
- note added: "步进绕组电流不等于电池输入电流；核对外置驱动模块 VM 范围和本地电容。"
- note added: "注意：本图未实现单节电压监测和欠压硬关断，须另设均衡监测与安全停机策略。"
- title: (none) -> EdgeMind 机器人 3S 电源控制板
