File: pcb/power/kicad/06_motor_right.kicad_sch (KiCad schematic)
At the start: 24 parts, among them J4 MG513 / verify harness, U11 74HC08D, U26 INA180A1IDBVR, U4 AT8236 dual module

Commit message: 10.3
Parts:
- removed F3: 3.15A, Fuse:Fuseholder_Clip-5x20mm_Littelfuse_100_Inline_P20.50x4.60mm_D1.30mm_Horizontal, symbol Device:Fuse
- J4: value MG513 / verify harness -> MG513电机 / 核对线序
- U4: value AT8236 dual module -> AT8236双路模块
Connections:
- net 电机总电源: now reaches R94.1, U26.3 (+)
- net +3V3 renamed 本板3.3V
- net +3V3_SENS renamed 传感器电源
- net ENC_R_A renamed 右编码器_A
- net ENC_R_A_FPGA renamed 右编码器_A_逻辑板输入
- net ENC_R_B renamed 右编码器_B
- net ENC_R_B_FPGA renamed 右编码器_B_逻辑板输入
- net GND renamed 地
- net MOTOR_ARMED renamed 已解锁
- net 已解锁: no longer U11.13
- net R_PWM_FWD_RAW renamed 正转脉宽
- net R_PWM_REV_RAW renamed 反转脉宽
- net VM_R renamed 右电机_动力电源
- net VM_R_IMON renamed 右电机_母线电流采样
- net VREF_R renamed 右电机_限流参考
- new net 电机已解锁: U11.13
Other:
- note added: "右电机驱动：使用A通道 / 可调限流参考 / 双排排母"
- note added: "右电机：电子过流关断、电流监测与本地储能"
- note added: "增益20，采样电阻20mΩ：约0.4V/A 输出滤波约1ms；母线过流阈值约3.04A 母线电流不同于绕组电流；滤波关断不能替代入口保护 入口总保险板载；模块内部限流须校准"
- note added: "排间距23.1275毫米，沿用原电路板；对排引脚编号已纠正。 限流电流=参考电压/(10×采样电阻)；安装电机前先测阻值并校准。 10正转、01反转、00滑行、11制动；B通道未用。编码器线序须与实物一致。"
- note removed: "Gain 20 / shunt 20mohm -> 0.4V/A 1ms output filter; bus current != winding current Fault threshold ~3.04A bus, needs bench setting"
- note removed: "R AT8236 / A channel / VREF adjustable / female sockets"
- note removed: "R MOTOR / branch fuse / bus current monitor / local bulk"
- note removed: "ROW=23.1275mm, from existing PCB. Opposing row numbering corrected. Itrip=VREF/(10 x Rsense); measure module Rsense and calibrate before fitting motors. 10=FWD / 01=REV / 00=coast / 11=brake. B unused. Encoder type/pinout must match harness."
- company: EdgeMind Robot -> EdgeMind机器人
- title: Right AT8236 and current monitor -> 右电机驱动与电流监测
- moved on the sheet: R98, R99

Commit message: 10.3
Connections:
- net 电机已解锁 is gone; now on net MOTOR_ARMED: U11.13
- net 传感器电源 renamed +3V3_SENS
- net 反转脉宽 renamed R_PWM_REV_RAW
- net 右电机_动力电源 renamed VM_R
- net 右电机_母线电流采样 renamed VM_R_IMON
- net 右电机_限流参考 renamed VREF_R
- net 右编码器_A renamed ENC_R_A
- net 右编码器_A_逻辑板输入 renamed ENC_R_A_FPGA
- net 右编码器_B renamed ENC_R_B
- net 右编码器_B_逻辑板输入 renamed ENC_R_B_FPGA
- net 地 renamed GND
- net 已解锁 renamed MOTOR_ARMED
- net 本板3.3V renamed +3V3
- net 正转脉宽 renamed R_PWM_FWD_RAW
- net 电机总电源 renamed VM_SWITCHED
Changed lines of the file:
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@@
 	(wire
 		(pts
-			(xy 104.14 217.17) (xy 96.52 217.17)
+			(xy 104.14 217.17) (xy 78.74 217.17)
 		)
 		(stroke
@@
 		)
 	)
-	(global_label "右电机_动力电源"
+	(global_label "VM_R"
 		(shape passive)
 		(at 220.98 161.29 0)
@@
 		)
 	)
-	(global_label "右编码器_B"
+	(global_label "ENC_R_B"
 		(shape passive)
 		(at 281.94 194.31 180)
@@
 		)
 	)
-	(global_label "本板3.3V"
+	(global_label "+3V3"
 		(shape passive)
 		(at 200.66 218.44 0)
@@
 		)
 	)
-	(global_label "本板3.3V"
+	(global_label "+3V3"
 		(shape passive)
 		(at 195.58 95.25 0)
@@
 		)
 	)
-	(global_label "右电机_动力电源"
+	(global_label "VM_R"
 		(shape passive)
 		(at 254 50.8 0)
@@
 		)
 	)
-	(global_label "本板3.3V"
+	(global_label "+3V3"
 		(shape passive)
 		(at 281.94 189.23 180)
@@
 		)
 	)
-	(global_label "右电机_限流参考"
+	(global_label "VREF_R"
 		(shape passive)
 		(at 181.61 147.32 0)
@@
 		)
 	)
-	(global_label "右编码器_A"
+	(global_label "ENC_R_A"
 		(shape passive)
 		(at 48.26 238.76 180)
@@
 		)
 	)
-	(global_label "本板3.3V"
+	(global_label "+3V3"
 		(shape passive)
 		(at 91.44 218.44 0)
@@
 		)
 	)
-	(global_label "右编码器_B_逻辑板输入"
+	(global_label "ENC_R_B_FPGA"
 		(shape passive)
 		(at 177.8 238.76 0)
@@
 		)
 	)
-	(global_label "地"
+	(global_label "GND"
 		(shape passive)
 		(at 281.94 196.85 180)
@@
 		)
 	)
-	(global_label "右编码器_B"
+	(global_label "ENC_R_B"
 		(shape passive)
 		(at 157.48 238.76 180)
@@
 		)
 	)
-	(global_label "右编码器_A_逻辑板输入"
+	(global_label "ENC_R_A_FPGA"
 		(shape passive)
 		(at 68.58 238.76 0)
@@
 		)
 	)
-	(global_label "右编码器_A"
+	(global_label "ENC_R_A"
 		(shape passive)
 		(at 281.94 191.77 180)
@@
 		)
 	)
-	(global_label "本板3.3V"
+	(global_label "+3V3"
 		(shape passive)
 		(at 342.9 180.34 0)
@@
 		)
 	)
-	(global_label "电机已解锁"
+	(global_label "MOTOR_ARMED"
 		(shape passive)
-		(at 96.52 217.17 180)
+		(at 78.74 217.17 180)
 		(effects
 			(font
@@
 		)
 		(property "Intersheetrefs" "${INTERSHEET_REFS}"
-			(at 96.52 217.17 180)
+			(at 78.74 217.17 180)
 			(hide yes)
 			(show_name no)
@@
 		)
 	)
-	(global_label "右电机_母线电流采样"
+	(global_label "VM_R_IMON"
 		(shape passive)
 		(at 209.55 81.28 0)
@@
 		)
 	)
-	(hierarchical_label "电机总电源"
+	(hierarchical_label "VM_SWITCHED"
 		(shape passive)
 		(at 34.29 50.8 180)
@@
 		)
 	)
-	(hierarchical_label "反转脉宽"
+	(hierarchical_label "R_PWM_REV_RAW"
 		(shape passive)
 		(at 96.52 212.09 180)
@@
 		)
 	)
-	(hierarchical_label "传感器电源"
+	(hierarchical_label "+3V3_SENS"
 		(shape passive)
 		(at 132.08 139.7 0)
@@
 		)
 	)
-	(hierarchical_label "正转脉宽"
+	(hierarchical_label "R_PWM_FWD_RAW"
 		(shape passive)
 		(at 96.52 186.69 180)
@@
 		)
 	)
-	(hierarchical_label "已解锁"
+	(hierarchical_label "MOTOR_ARMED"
 		(shape passive)
 		(at 96.52 191.77 180)
@@
 		)
 	)
-	(hierarchical_label "本板3.3V"
+	(hierarchical_label "+3V3"
 		(shape passive)
 		(at 154.94 69.85 0)
@@
 			)
 		)
-		(property "Value" "地"
+		(property "Value" "GND"
 			(at 199.39 153.67 0)
 			(hide yes)
@@
 			)
 		)
-		(property "Value" "地"
+		(property "Value" "GND"
 			(at 342.9 179.07 0)
 			(hide yes)
@@
 			)
 		)
-		(property "Value" "地"
+		(property "Value" "GND"
 			(at 246.38 64.77 0)
 			(hide yes)
@@
 			)
 		)
-		(property "Value" "地"
+		(property "Value" "GND"
 			(at 147.32 219.71 0)
 			(hide yes)
@@
 			)
 		)
-		(property "Value" "地"
+		(property "Value" "GND"
 			(at 195.58 93.98 0)
 			(hide yes)
@@
 			)
 		)
-		(property "Value" "地"
+		(property "Value" "GND"
 			(at 220.98 196.85 0)
 			(hide yes)
@@
 			)
 		)
-		(property "Value" "地"
+		(property "Value" "GND"
 			(at 177.8 242.57 0)
 			(hide yes)
@@
 			)
 		)
-		(property "Value" "地"
+		(property "Value" "GND"
 			(at 132.08 138.43 0)
 			(hide yes)
@@
 			)
 		)
-		(property "Value" "地"
+		(property "Value" "GND"
 			(at 200.66 181.61 0)
 			(hide yes)
@@
 			)
 		)
-		(property "Value" "地"
+		(property "Value" "GND"
 			(at 181.61 153.67 0)
 			(hide yes)
@@
 			)
 		)
-		(property "Value" "地"
+		(property "Value" "GND"
 			(at 226.06 64.77 0)
 			(hide yes)
@@
 			)
 		)
-		(property "Value" "地"
+		(property "Value" "GND"
 			(at 160.02 194.31 0)
 			(hide yes)
@@
 			)
 		)
-		(property "Value" "地"
+		(property "Value" "GND"
 			(at 68.58 242.57 0)
 			(hide yes)
@@
 			)
 		)
-		(property "Value" "地"
+		(property "Value" "GND"
 			(at 154.94 76.2 0)
 			(hide yes)
@@
 			)
 		)
-		(property "Value" "地"
+		(property "Value" "GND"
 			(at 209.55 87.63 0)
 			(hide yes)
