File: pcb/power/kicad/07_motor_dump.kicad_sch (KiCad schematic)
At the start: 22 parts, among them J16 L DUMP / external 3R3, J17 R DUMP / external 3R3, Q2 IRF4905, Q5 MMBT3904, Q6 IRLZ44N, Q7 IRLZ44N, U24 LM393BIDR

Commit message: 10.3
Parts:
- J16: value L DUMP / external 3R3 -> 左回生泄放 / 外接3.3Ω
- J17: value R DUMP / external 3R3 -> 右回生泄放 / 外接3.3Ω
- TP1: value VM_SWITCHED -> 电机总开关输出
Connections:
- net GND renamed 地
- net 地: no longer R76.2, R77.1, R79.1, R80.2, R81.1, R83.1, U24.3 (+), U24.5 (+)
- net MOTOR_ARMED renamed 已解锁
- net VBAT_SYS renamed 电池保护后母线
- net 电池保护后母线: no longer Q2.3 (S)
- net VM_L renamed 左电机_动力电源
- net VM_R renamed 右电机_动力电源
- net VM_SWITCHED renamed 电机总开关输出
- net 电机总开关输出: no longer Q2.2 (D)
- net VREF_2V495 renamed 基准电压_2.495V
- new net: R76.2, R77.1, R79.1, U24.3 (+)
- new net: R80.2, R81.1, R83.1, U24.5 (+)
- new net 电机总电源: Q2.2 (D)
- new net 电池母线: Q2.3 (S)
Other:
- note added: "动力总开关 / 急停触点只承载控制电流"
- note added: "回生能量泄放 / 外接底盘散热电阻"
- note added: "约15.39V开始泄放；关闭阈值和最坏过冲须实测。 若电源或电池保护板不能吸收回生，外接两只3.3Ω、至少100W的底盘散热电阻。 电路由电池母线供电，本板3.3V消失时仍可工作；功率管需要散热。"
- note removed: "Dump turns ON ~15.39V; verify OFF threshold and worst-case overshoot. Use two 3.3ohm >=100W chassis resistors if the supply/BMS cannot absorb regen. Circuit operates from raw bus even when local 3V3 is absent. MOSFET cooling required."
- note removed: "MOTOR POWER SWITCH / not a small slider in the motor path"
- note removed: "REGEN DUMP / external chassis resistors"
- company: EdgeMind Robot -> EdgeMind机器人
- title: Regeneration dump -> 电机回生能量泄放

Commit message: 10.3
Connections:
- net 电机总电源 is gone; now on net VM_SWITCHED: Q2.2 (D)
- net 电池母线 is gone; now on net VBAT_SYS: Q2.3 (S)
- net 右电机_动力电源 renamed VM_R
- net 地 renamed GND
- net 基准电压_2.495V renamed VREF_2V495
- net 左电机_动力电源 renamed VM_L
- net 已解锁 renamed MOTOR_ARMED
- net 电机总开关输出 renamed VM_SWITCHED
- net 电池保护后母线 renamed VBAT_SYS
Changed lines of the file:
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@@
 		)
 	)
-	(global_label "基准电压_2.495V"
+	(global_label "VREF_2V495"
 		(shape passive)
 		(at 251.46 66.04 180)
@@
 		)
 	)
-	(global_label "右电机_动力电源"
+	(global_label "VM_R"
 		(shape passive)
 		(at 224.79 146.05 0)
@@
 		)
 	)
-	(global_label "右电机_动力电源"
+	(global_label "VM_R"
 		(shape passive)
 		(at 302.26 142.24 0)
@@
 		)
 	)
-	(global_label "右电机_动力电源"
+	(global_label "VM_R"
 		(shape passive)
 		(at 375.92 152.4 180)
@@
 		)
 	)
-	(global_label "电机总开关输出"
+	(global_label "VM_SWITCHED"
 		(shape passive)
 		(at 43.18 119.38 0)
@@
 		)
 	)
-	(global_label "电池保护后母线"
+	(global_label "VBAT_SYS"
 		(shape passive)
 		(at 81.28 39.37 0)
@@
 		)
 	)
-	(global_label "电池保护后母线"
+	(global_label "VBAT_SYS"
 		(shape passive)
 		(at 241.3 227.33 0)
@@
 		)
 	)
-	(global_label "基准电压_2.495V"
+	(global_label "VREF_2V495"
 		(shape passive)
 		(at 251.46 170.18 180)
@@
 		)
 	)
-	(global_label "左电机_动力电源"
+	(global_label "VM_L"
 		(shape passive)
 		(at 375.92 48.26 180)
@@
 		)
 	)
-	(global_label "左电机_动力电源"
+	(global_label "VM_L"
 		(shape passive)
 		(at 224.79 41.91 0)
@@
 		)
 	)
-	(global_label "电池保护后母线"
+	(global_label "VBAT_SYS"
 		(shape passive)
 		(at 96.52 74.93 0)
@@
 		)
 	)
-	(global_label "左电机_动力电源"
+	(global_label "VM_L"
 		(shape passive)
 		(at 302.26 38.1 0)
@@
 		)
 	)
-	(global_label "电机总开关输出"
+	(global_label "VM_SWITCHED"
 		(shape passive)
 		(at 158.75 123.19 0)
@@
 		)
 	)
-	(hierarchical_label "电机总电源"
+	(hierarchical_label "VM_SWITCHED"
 		(shape passive)
 		(at 121.92 60.96 0)
@@
 		)
 	)
-	(hierarchical_label "已解锁"
+	(hierarchical_label "MOTOR_ARMED"
 		(shape passive)
 		(at 46.99 99.06 180)
@@
 		)
 	)
-	(hierarchical_label "电池母线"
+	(hierarchical_label "VBAT_SYS"
 		(shape passive)
 		(at 96.52 60.96 180)
@@
 			)
 		)
-		(property "Value" "地"
+		(property "Value" "GND"
 			(at 224.79 170.18 0)
 			(hide yes)
@@
 			)
 		)
-		(property "Value" "地"
+		(property "Value" "GND"
 			(at 312.42 74.93 0)
 			(hide yes)
@@
 			)
 		)
-		(property "Value" "地"
+		(property "Value" "GND"
 			(at 335.28 55.88 0)
 			(hide yes)
@@
 			)
 		)
-		(property "Value" "地"
+		(property "Value" "GND"
 			(at 312.42 179.07 0)
 			(hide yes)
@@
 			)
 		)
-		(property "Value" "地"
+		(property "Value" "GND"
 			(at 261.62 237.49 0)
 			(hide yes)
@@
 			)
 		)
-		(property "Value" "地"
+		(property "Value" "GND"
 			(at 81.28 91.44 0)
 			(hide yes)
@@
 			)
 		)
-		(property "Value" "地"
+		(property "Value" "GND"
 			(at 224.79 66.04 0)
 			(hide yes)
@@
 			)
 		)
-		(property "Value" "地"
+		(property "Value" "GND"
 			(at 335.28 160.02 0)
 			(hide yes)
