File: pcb/power/kicad/01_power_input.kicad_sch (KiCad schematic)
At the start: 31 parts, among them CN1 XT60PW-M / 3S, Q1 IRF4905, Q3 IRF4905, Q4 MMBT3904, U21 TL431BIDBZR, U22 LM393BIDR, U23 LM393BIDR

Commit message: 10.3
Parts:
- CN1: value XT60PW-M / 3S -> XT60PW-M / 三串电池
- F1: value 10A -> 10A/32V MINI总保险; footprint Fuse:Fuseholder_Blade_ATO_Littelfuse_Pudenz_2_Pin -> Fuse:Fuseholder_Blade_Mini_Keystone_3568; MPN (none) -> 0297010.J; Specification 10A 32VDC ATO (initial) -> MINI汽车插片保险丝10A/32VDC；初值须实测；保险座四孔9.92×3.40mm、钻孔1.78mm; 供应商编号 (none) -> C55117678; 保险座供应商编号 (none) -> C5249699（立创查询时缺货，可核对其他渠道）; 保险座参考链接 (none) -> https://www.digikey.cn/zh/products/detail/keystone-electron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; 保险座型号 (none) -> 3568 / 同四孔尺寸兼容品待核对; 保险座数据手册 (none) -> https://www.keyelco.com/product-pdf.cfm?p=306; 安装位置 (none) -> 板上，XT60正极之后、防反接管之前; 购买链接 (none) -> https://www.lcsc.com/pt/product-detail/C55117678.html?is_su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
Connections:
- net 电池正极: now reaches CN1.2 (Pin_2), F1.1
- net +3V3 renamed 本板3.3V
- net BUCK_ENABLE renamed 降压使能
- net 降压使能: no longer R54.1
- net GND renamed 地
- net MOTOR_POWER_OK renamed 电机供电正常
- net 电机供电正常: no longer U23.1
- net VBAT_SYS renamed 电池保护后母线
- net 电池保护后母线: no longer C58.1, C59.1, C60.1, D1.1 (A1), D2.1 (K), Q1.3 (S)
- net VLOGIC_IN renamed 降压电源输入
- net 降压电源输入: no longer Q3.2 (D)
- net VREF_2V495 renamed 基准电压_2.495V
- new net 使能: R54.1
- new net 动力正常: U23.1
- new net 电池母线: C58.1, C59.1, C60.1, D1.1 (A1), D2.1 (K), Q1.3 (S)
- new net 降压输入: Q3.2 (D)
Other:
- note added: "开集电极故障输出共同拉低使能。电机故障清除解锁锁存；电压恢复后不自动解锁。 总电压监测不能替代单体电芯保护。阈值、响应和过冲须实测。"
- note added: "欠压与过压窗口：逻辑约9.0-14.1V；动力约9.65-14.1V"
- note added: "电池母线基准与降压输入开关"
- note added: "电池：11.1V / 3600mAh / 35C；满电12.6V。 F1板载：XT60正极之后、防反接管之前。 保险片：集电通0297010.J，10A/32V，初值待实测。 保险座：四孔9.92×3.40mm；与保险片分别采购。 照片不能确认电池保护板；单体电芯保护仍须落实。 瞬态抑制二极管不能把电压固定在17V以下。"
- note added: "输入：三串11.1V锂聚合物电池 / 板载总保险与防反接"
- note removed: "INPUT / 3S pack + external BMS / fuse + reverse polarity"
- note removed: "OC outputs wired-AND. Motor faults clear the arm latch; voltage recovery does not re-arm. Total voltage monitoring does not replace cell protection. Validate threshold/overshoot on bench."
- note removed: "Q1: D=BAT input / S=VBAT_SYS TVS handles transients, not a 17V clamp. Fuse rating must match copper and harness."
- note removed: "RAW-BUS reference / logic input switch"
- note removed: "UV / OV WINDOW: logic 9.0-14.1V, motor 9.65-14.1V"
- company: EdgeMind Robot -> EdgeMind机器人
- title: 3S input and voltage protection -> 三串电池输入与电压保护

Commit message: 10.3
Connections:
- net 电机供电正常 is gone; now on net MOTOR_POWER_OK: R64.2, U23.7
- net 电池母线 is gone; now on net VBAT_SYS: C58.1, C59.1, C60.1, D1.1 (A1), D2.1 (K), Q1.3 (S)
- net 降压使能 is gone; now on net BUCK_ENABLE: R59.2, U22.1, U22.7
- net 降压输入 is gone; now on net VLOGIC_IN: Q3.2 (D)
- net 使能 renamed BUCK_ENABLE
- net 动力正常 renamed MOTOR_POWER_OK
- net 地 renamed GND
- net 基准电压_2.495V renamed VREF_2V495
- net 本板3.3V renamed +3V3
- net 电池保护后母线 renamed VBAT_SYS
- net 电池正极 renamed BAT_POS
- net 降压电源输入 renamed VLOGIC_IN
Changed lines of the file:
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@@
 		)
 	)
-	(label "电池正极"
+	(global_label "BAT_POS" (shape passive)
 		(at 50.8 52.07 0)
 		(effects
@@
 		)
 	)
-	(global_label "地"
+	(global_label "GND"
 		(shape passive)
 		(at 35.56 58.42 0)
@@
 		)
 	)
-	(global_label "降压使能"
+	(global_label "BUCK_ENABLE"
 		(shape passive)
 		(at 276.86 229.87 0)
@@
 		)
 	)
-	(global_label "基准电压_2.495V"
+	(global_label "VREF_2V495"
 		(shape passive)
 		(at 335.28 201.93 180)
@@
 		)
 	)
-	(global_label "电机供电正常"
+	(global_label "MOTOR_POWER_OK"
 		(shape passive)
 		(at 360.68 247.65 0)
@@
 		)
 	)
-	(global_label "电机供电正常"
+	(global_label "MOTOR_POWER_OK"
 		(shape passive)
 		(at 365.76 204.47 0)
@@
 		)
 	)
-	(global_label "基准电压_2.495V"
+	(global_label "VREF_2V495"
 		(shape passive)
 		(at 335.28 149.86 180)
@@
 		)
 	)
-	(global_label "电池保护后母线"
+	(global_label "VBAT_SYS"
 		(shape passive)
 		(at 222.25 129.54 0)
@@
 		)
 	)
-	(global_label "电池保护后母线"
+	(global_label "VBAT_SYS"
 		(shape passive)
 		(at 104.14 143.51 0)
@@
 		)
 	)
-	(global_label "电池保护后母线"
+	(global_label "VBAT_SYS"
 		(shape passive)
 		(at 307.34 229.87 0)
@@
 		)
 	)
-	(global_label "电池保护后母线"
+	(global_label "VBAT_SYS"
 		(shape passive)
 		(at 119.38 165.1 180)
@@
 		)
 	)
-	(global_label "降压电源输入"
+	(global_label "VLOGIC_IN"
 		(shape passive)
 		(at 157.48 233.68 0)
@@
 		)
 	)
-	(global_label "电池保护后母线"
+	(global_label "VBAT_SYS"
 		(shape passive)
 		(at 222.25 181.61 0)
@@
 		)
 	)
-	(global_label "本板3.3V"
+	(global_label "+3V3"
 		(shape passive)
 		(at 360.68 232.41 0)
@@
 		)
 	)
-	(global_label "电池保护后母线"
+	(global_label "VBAT_SYS"
 		(shape passive)
 		(at 240.03 222.25 0)
@@
 		)
 	)
-	(global_label "电池保护后母线"
+	(global_label "VBAT_SYS"
 		(shape passive)
 		(at 119.38 179.07 0)
@@
 		)
 	)
-	(global_label "降压电源输入"
+	(global_label "VLOGIC_IN"
 		(shape passive)
 		(at 172.72 233.68 0)
@@
 		)
 	)
-	(global_label "电池保护后母线"
+	(global_label "VBAT_SYS"
 		(shape passive)
 		(at 276.86 214.63 0)
@@
 		)
 	)
-	(global_label "基准电压_2.495V"
+	(global_label "VREF_2V495"
 		(shape passive)
 		(at 53.34 146.05 0)
@@
 		)
 	)
-	(global_label "降压使能"
+	(global_label "BUCK_ENABLE"
 		(shape passive)
 		(at 275.59 152.4 0)
@@
 		)
 	)
-	(global_label "基准电压_2.495V"
+	(global_label "VREF_2V495"
 		(shape passive)
 		(at 245.11 154.94 180)
@@
 		)
 	)
-	(global_label "电池保护后母线"
+	(global_label "VBAT_SYS"
 		(shape passive)
 		(at 312.42 186.69 0)
@@
 		)
 	)
-	(global_label "降压使能"
+	(global_label "BUCK_ENABLE"
 		(shape passive)
 		(at 365.76 152.4 0)
@@
 		)
 	)
-	(global_label "基准电压_2.495V"
+	(global_label "VREF_2V495"
 		(shape passive)
 		(at 245.11 207.01 180)
@@
 		)
 	)
-	(global_label "电池保护后母线"
+	(global_label "VBAT_SYS"
 		(shape passive)
 		(at 53.34 125.73 0)
@@
 		)
 	)
-	(global_label "电池保护后母线"
+	(global_label "VBAT_SYS"
 		(shape passive)
 		(at 312.42 134.62 0)
@@
 		)
 	)
-	(hierarchical_label "降压输入"
+	(hierarchical_label "VLOGIC_IN"
 		(shape passive)
 		(at 144.78 165.1 0)
@@
 		)
 	)
-	(hierarchical_label "使能"
+	(hierarchical_label "BUCK_ENABLE"
 		(shape passive)
 		(at 69.85 203.2 180)
@@
 		)
 	)
-	(hierarchical_label "电池母线"
+	(hierarchical_label "VBAT_SYS"
 		(shape passive)
 		(at 187.96 63.5 0)
@@
 		)
 	)
-	(hierarchical_label "动力正常"
+	(hierarchical_label "MOTOR_POWER_OK"
 		(shape passive)
 		(at 275.59 204.47 0)
@@
 			)
 		)
-		(property "Value" "地"
+		(property "Value" "GND"
 			(at 35.56 41.91 0)
 			(hide yes)
@@
 			)
 		)
-		(property "Value" "地"
+		(property "Value" "GND"
 			(at 260.35 232.41 0)
 			(hide yes)
@@
 			)
 		)
-		(property "Value" "地"
+		(property "Value" "GND"
 			(at 312.42 158.75 0)
 			(hide yes)
@@
 			)
 		)
-		(property "Value" "地"
+		(property "Value" "GND"
 			(at 222.25 205.74 0)
 			(hide yes)
@@
 			)
 		)
-		(property "Value" "地"
+		(property "Value" "GND"
 			(at 246.38 57.15 0)
 			(hide yes)
@@
 			)
 		)
-		(property "Value" "地"
+		(property "Value" "GND"
 			(at 222.25 153.67 0)
 			(hide yes)
@@
 			)
 		)
-		(property "Value" "地"
+		(property "Value" "GND"
 			(at 327.66 240.03 0)
 			(hide yes)
@@
 			)
 		)
-		(property "Value" "地"
+		(property "Value" "GND"
 			(at 157.48 232.41 0)
 			(hide yes)
@@
 			)
 		)
-		(property "Value" "地"
+		(property "Value" "GND"
 			(at 205.74 57.15 0)
 			(hide yes)
@@
 			)
 		)
-		(property "Value" "地"
+		(property "Value" "GND"
 			(at 53.34 138.43 0)
 			(hide yes)
@@
 			)
 		)
-		(property "Value" "地"
+		(property "Value" "GND"
 			(at 104.14 195.58 0)
 			(hide yes)
@@
 			)
 		)
-		(property "Value" "地"
+		(property "Value" "GND"
 			(at 111.76 76.2 0)
 			(hide yes)
@@
 			)
 		)
-		(property "Value" "地"
+		(property "Value" "GND"
 			(at 269.24 57.15 0)
 			(hide yes)
@@
 			)
 		)
-		(property "Value" "地"
+		(property "Value" "GND"
 			(at 226.06 57.15 0)
 			(hide yes)
@@
 			)
 		)
-		(property "Value" "地"
+		(property "Value" "GND"
 			(at 312.42 210.82 0)
 			(hide yes)

Commit message: 10.4
Other:
- moved on the sheet: C101, C103, D3, Q3, Q4, R52, R53, R54, R55, R56, R62, R63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
