File: pcb/power/kicad/02_usb_5v.kicad_sch (KiCad schematic)
At the start: 38 parts, among them U1 MP2236GJ-Z, U5 MP2236GJ-Z, U7 HUSB305-02, U8 HUSB305-02

Commit message: 10.3
Parts:
- USB1, USB2: value TYPE-C-31-M-17 / 6P -> USB4125-GF-A / 六针供电; footprint Connector_USB:USB_C_Receptacle_HRO_TYPE-C-31-M-17 -> Connector_USB:USB_C_Receptacle_GCT_USB4125-xx-x_6P_TopMnt_Horizontal; MPN TYPE-C-31-M-17 -> USB4125-GF-A
Connections:
- net +3V3 renamed 本板3.3V
- net +5V_AI renamed 计算5V
- net +5V_AI_PROT renamed 计算5V保护
- net +5V_FPGA renamed 逻辑5V
- net +5V_FPGA_PROT renamed 逻辑5V保护
- net BUCK_ENABLE renamed 使能
- net 使能: no longer U1.6 (EN)
- net GND renamed 地
- net USB1_FAULT_PULSE_N renamed 供电口1_故障脉冲_低有效
- net USB1_VBUS renamed 供电口1_总线电源
- net USB2_FAULT_PULSE_N renamed 供电口2_故障脉冲_低有效
- net USB2_VBUS renamed 供电口2_总线电源
- net VLOGIC_IN renamed 降压电源输入
- net 降压电源输入: no longer C1.1, C2.1, C3.1, U5.2 (IN)
- new net 降压使能: U1.6 (EN)
- new net 降压输入: C1.1, C2.1, C3.1, U5.2 (IN)
Other:
- note added: "USB1 / 六针供电口 / 固定5V"
- note added: "USB2 / 六针供电口 / 固定5V"
- note added: "计算板5V_稳压输出 / 5.10V / 供电目标3A"
- note added: "连接检测与总线电源开关由控制器完成 限流电阻150kΩ：典型限流3.6A，宣告供电能力3A 无需外部上拉电阻；仅固定5V供电"
- note added: "逻辑板5V_稳压输出 / 5.10V / 供电目标3A"
- note removed: "+5V_AI / 5.10V / USB-C 3A target"
- note removed: "+5V_FPGA / 5.10V / USB-C 3A target"
- note removed: "CC attach detection + integrated VBUS switch ISET 150k: 3.6A typ / Rp advertises 3A No external Rp, USB data or PD voltage negotiation"
- note removed: "USB1 / 6P power-only / fixed 5V"
- note removed: "USB2 / 6P power-only / fixed 5V"
- company: EdgeMind Robot -> EdgeMind机器人
- title: Two MP2236 / 6P USB-C sources -> 两路5V降压与六针供电口

Commit message: 10.3
Connections:
- net 降压使能 is gone; now on net BUCK_ENABLE: U1.6 (EN)
- net 降压输入 is gone; now on net VLOGIC_IN: C1.1, C2.1, C3.1, U5.2 (IN)
- net 使能 renamed BUCK_ENABLE
- net 供电口1_总线电源 renamed USB1_VBUS
- net 供电口1_故障脉冲_低有效 renamed USB1_FAULT_PULSE_N
- net 供电口2_总线电源 renamed USB2_VBUS
- net 供电口2_故障脉冲_低有效 renamed USB2_FAULT_PULSE_N
- net 地 renamed GND
- net 本板3.3V renamed +3V3
- net 计算5V renamed +5V_AI
- net 计算5V保护 renamed +5V_AI_PROT
- net 逻辑5V renamed +5V_FPGA
- net 逻辑5V保护 renamed +5V_FPGA_PROT
- net 降压电源输入 renamed VLOGIC_IN
Other:
- note added: "计算板降压输出 / 5.10V / 供电目标3A"
- note added: "逻辑板降压输出 / 5.10V / 供电目标3A"
- note removed: "计算板5V_稳压输出 / 5.10V / 供电目标3A"
- note removed: "逻辑板5V_稳压输出 / 5.10V / 供电目标3A"
Changed lines of the file:
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@@
 		)
 	)
-	(text "逻辑板5V_稳压输出 / 5.10V / 供电目标3A"
+	(text "逻辑板降压输出 / 5.10V / 供电目标3A"
 		(exclude_from_sim no)
 		(at 18 34.21 0)
@@
 		)
 	)
-	(text "计算板5V_稳压输出 / 5.10V / 供电目标3A"
+	(text "计算板降压输出 / 5.10V / 供电目标3A"
 		(exclude_from_sim no)
 		(at 18 147.24 0)
@@
 		)
 	)
-	(global_label "供电口1_总线电源"
+	(global_label "USB1_VBUS"
 		(shape passive)
 		(at 312.42 64.77 0)
@@
 		)
 	)
-	(global_label "供电口2_故障脉冲_低有效"
+	(global_label "USB2_FAULT_PULSE_N"
 		(shape passive)
 		(at 302.26 198.12 0)
@@
 		)
 	)
-	(global_label "供电口2_总线电源"
+	(global_label "USB2_VBUS"
 		(shape passive)
 		(at 312.42 177.8 0)
@@
 		)
 	)
-	(global_label "供电口2_故障脉冲_低有效"
+	(global_label "USB2_FAULT_PULSE_N"
 		(shape passive)
 		(at 347.98 229.87 0)
@@
 		)
 	)
-	(global_label "本板3.3V"
+	(global_label "+3V3"
 		(shape passive)
 		(at 347.98 214.63 0)
@@
 		)
 	)
-	(global_label "降压电源输入"
+	(global_label "VLOGIC_IN"
 		(shape passive)
 		(at 35.56 177.8 180)
@@
 		)
 	)
-	(global_label "本板3.3V"
+	(global_label "+3V3"
 		(shape passive)
 		(at 347.98 101.6 0)
@@
 		)
 	)
-	(global_label "供电口1_故障脉冲_低有效"
+	(global_label "USB1_FAULT_PULSE_N"
 		(shape passive)
 		(at 302.26 85.09 0)
@@
 		)
 	)
-	(global_label "降压使能"
+	(global_label "BUCK_ENABLE"
 		(shape passive)
 		(at 63.5 185.42 180)
@@
 		)
 	)
-	(global_label "供电口1_故障脉冲_低有效"
+	(global_label "USB1_FAULT_PULSE_N"
 		(shape passive)
 		(at 347.98 116.84 0)
@@
 		)
 	)
-	(hierarchical_label "逻辑5V保护"
+	(hierarchical_label "+5V_FPGA_PROT"
 		(shape passive)
 		(at 243.84 64.77 0)
@@
 		)
 	)
-	(hierarchical_label "使能"
+	(hierarchical_label "BUCK_ENABLE"
 		(shape passive)
 		(at 63.5 72.39 180)
@@
 		)
 	)
-	(hierarchical_label "计算5V"
+	(hierarchical_label "+5V_AI"
 		(shape passive)
 		(at 205.74 177.8 0)
@@
 		)
 	)
-	(hierarchical_label "计算5V保护"
+	(hierarchical_label "+5V_AI_PROT"
 		(shape passive)
 		(at 243.84 177.8 0)
@@
 		)
 	)
-	(hierarchical_label "逻辑5V"
+	(hierarchical_label "+5V_FPGA"
 		(shape passive)
 		(at 205.74 64.77 0)
@@
 		)
 	)
-	(hierarchical_label "降压输入"
+	(hierarchical_label "VLOGIC_IN"
 		(shape passive)
 		(at 35.56 64.77 180)
@@
 			)
 		)
-		(property "Value" "地"
+		(property "Value" "GND"
 			(at 205.74 83.82 0)
 			(hide yes)
@@
 			)
 		)
-		(property "Value" "地"
+		(property "Value" "GND"
 			(at 165.1 207.01 0)
 			(hide yes)
@@
 			)
 		)
-		(property "Value" "地"
+		(property "Value" "GND"
 			(at 251.46 203.2 0)
 			(hide yes)
@@
 			)
 		)
-		(property "Value" "地"
+		(property "Value" "GND"
 			(at 360.68 26.67 0)
 			(hide yes)
@@
 			)
 		)
-		(property "Value" "地"
+		(property "Value" "GND"
 			(at 368.3 139.7 0)
 			(hide yes)
@@
 			)
 		)
-		(property "Value" "地"
+		(property "Value" "GND"
 			(at 35.56 95.25 0)
 			(hide yes)
@@
 			)
 		)
-		(property "Value" "地"
+		(property "Value" "GND"
 			(at 251.46 90.17 0)
 			(hide yes)
@@
 			)
 		)
-		(property "Value" "地"
+		(property "Value" "GND"
 			(at 38.1 179.07 0)
 			(hide yes)
@@
 			)
 		)
-		(property "Value" "地"
+		(property "Value" "GND"
 			(at 360.68 139.7 0)
 			(hide yes)
@@
 			)
 		)
-		(property "Value" "地"
+		(property "Value" "GND"
 			(at 63.5 66.04 0)
 			(hide yes)
@@
 			)
 		)
-		(property "Value" "地"
+		(property "Value" "GND"
 			(at 193.04 196.85 0)
 			(hide yes)
@@
 			)
 		)
-		(property "Value" "地"
+		(property "Value" "GND"
 			(at 312.42 203.2 0)
 			(hide yes)
@@
 			)
 		)
-		(property "Value" "地"
+		(property "Value" "GND"
 			(at 193.04 83.82 0)
 			(hide yes)
@@
 			)
 		)
-		(property "Value" "地"
+		(property "Value" "GND"
 			(at 312.42 90.17 0)
 			(hide yes)
@@
 			)
 		)
-		(property "Value" "地"
+		(property "Value" "GND"
 			(at 50.8 179.07 0)
 			(hide yes)
@@
 			)
 		)
-		(property "Value" "地"
+		(property "Value" "GND"
 			(at 279.4 193.04 0)
 			(hide yes)
@@
 			)
 		)
-		(property "Value" "地"
+		(property "Value" "GND"
 			(at 63.5 179.07 0)
 			(hide yes)
@@
 			)
 		)
-		(property "Value" "地"
+		(property "Value" "GND"
 			(at 205.74 196.85 0)
 			(hide yes)
@@
 			)
 		)
-		(property "Value" "地"
+		(property "Value" "GND"
 			(at 165.1 93.98 0)
 			(hide yes)
@@
 			)
 		)
-		(property "Value" "地"
+		(property "Value" "GND"
 			(at 50.8 66.04 0)
 			(hide yes)
@@
 			)
 		)
-		(property "Value" "地"
+		(property "Value" "GND"
 			(at 243.84 68.58 0)
 			(hide yes)
@@
 			)
 		)
-		(property "Value" "地"
+		(property "Value" "GND"
 			(at 368.3 26.67 0)
 			(hide yes)
@@
 			)
 		)
-		(property "Value" "地"
+		(property "Value" "GND"
 			(at 243.84 181.61 0)
 			(hide yes)
@@
 			)
 		)
-		(property "Value" "地"
+		(property "Value" "GND"
 			(at 86.36 198.12 0)
 			(hide yes)
@@
 			)
 		)
-		(property "Value" "地"
+		(property "Value" "GND"
 			(at 86.36 85.09 0)
 			(hide yes)
@@
 			)
 		)
-		(property "Value" "地"
+		(property "Value" "GND"
 			(at 35.56 208.28 0)
 			(hide yes)
@@
 			)
 		)
-		(property "Value" "地"
+		(property "Value" "GND"
 			(at 279.4 80.01 0)
 			(hide yes)
@@
 			)
 		)
-		(property "Value" "地"
+		(property "Value" "GND"
 			(at 38.1 66.04 0)
 			(hide yes)

Commit message: 10.4
Other:
- moved on the sheet: C11
Changed lines of the file:
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@@
 		(effects
 			(font
-				(size 1.52 1.52)
+				(size 2.54 2.54)
 			)
 			(justify left)
@@
 		(effects
 			(font
-				(size 1.52 1.52)
+				(size 2.54 2.54)
 			)
 			(justify left)
@@
 		(effects
 			(font
-				(size 0.95 0.95)
+				(size 2.54 2.54)
 			)
 			(justify left)
@@
 		(effects
 			(font
-				(size 1 1)
+				(size 2.54 2.54)
 			)
 			(justify left)
@@
 		(effects
 			(font
-				(size 1.52 1.52)
+				(size 2.54 2.54)
 			)
 			(justify left)
@@
 		(effects
 			(font
-				(size 0.95 0.95)
+				(size 2.54 2.54)
 			)
 			(justify left)
@@
 		(effects
 			(font
-				(size 1.52 1.52)
+				(size 2.54 2.54)
 			)
 			(justify left)
@@
 	(wire
 		(pts
-			(xy 43.18 100.33) (xy 35.56 100.33)
-		)
-		(stroke
-			(width 0)
-			(type default)
-		)
-	)
-	(wire
-		(pts
 			(xy 86.36 97.79) (xy 86.36 101.6)
 		)
@@
 	(wire
 		(pts
-			(xy 35.56 107.95) (xy 35.56 111.76)
+			(xy 43.18 107.95) (xy 43.18 111.76)
 		)
 		(stroke
@@
 	(symbol
 		(lib_id "power:GND")
-		(at 35.56 111.76 0)
+		(at 43.18 111.76 0)
 		(unit 1)
 		(body_style 1)
@@
 		(dnp no)
 		(property "Reference" "#PWR119"
-			(at 35.56 92.71 0)
+			(at 43.18 92.71 0)
 			(hide yes)
 			(show_name no)
@@
 		)
 		(property "Value" "GND"
-			(at 35.56 95.25 0)
+			(at 43.18 95.25 0)
 			(hide yes)
 			(show_name no)
@@
 		)
 		(property "Footprint" ""
-			(at 35.56 109.22 0)
+			(at 43.18 109.22 0)
 			(hide yes)
 			(show_name no)
@@
 		)
 		(property "Datasheet" ""
-			(at 35.56 109.22 0)
+			(at 43.18 109.22 0)
 			(hide yes)
 			(show_name no)
@@
 		)
 		(property "Description" "Power symbol creates a global label with name \"GND\" , ground"
-			(at 35.56 109.22 0)
+			(at 43.18 109.22 0)
 			(hide yes)
 			(show_name no)
@@
 	(symbol
 		(lib_id "Device:C")
-		(at 35.56 104.14 0)
+		(at 43.18 104.14 0)
 		(unit 1)
 		(body_style 1)
@@
 		(dnp no)
 		(property "Reference" "C11"
-			(at 38.56 102.84 0)
+			(at 46.18 102.84 0)
 			(show_name no)
 			(do_not_autoplace no)
@@
 		)
 		(property "Value" "1uF/25V"
-			(at 38.56 105.44 0)
+			(at 46.18 105.44 0)
 			(show_name no)
 			(do_not_autoplace no)
@@
 		)
 		(property "Footprint" "Capacitor_SMD:C_0805_2012Metric"
-			(at 38.56 105.44 0)
+			(at 46.18 105.44 0)
 			(hide yes)
 			(show_name no)
@@
 		)
 		(property "Datasheet" ""
-			(at 38.56 105.44 0)
+			(at 46.18 105.44 0)
 			(hide yes)
 			(show_name no)
@@
 		)
 		(property "Description" "Unpolarized capacitor"
-			(at 38.56 105.44 0)
+			(at 46.18 105.44 0)
 			(hide yes)
 			(show_name no)
@@
 		)
 		(property "Specification" "1uF 25V"
-			(at 38.56 105.44 0)
+			(at 46.18 105.44 0)
 			(hide yes)
 			(show_name no)
