File: pcb/power/kicad/03_aux_3v3.kicad_sch (KiCad schematic)
At the start: 20 parts, among them J10 IMU PWR, J11 TOF1 PWR, J12 TOF2 PWR, J13 TOF3 PWR, J14 3V3 AUX OUT, J9 OPTIONAL FPGA 3V3 IN, U3 AP63203WU-7

Commit message: 10.3
Parts:
- FB1: value 220R@100MHz 1A -> 220Ω@100MHz / 1A
- J10: value IMU PWR -> 惯性传感器电源
- J11: value TOF1 PWR -> 测距传感器1电源
- J12: value TOF2 PWR -> 测距传感器2电源
- J13: value TOF3 PWR -> 测距传感器3电源
- J14: value 3V3 AUX OUT -> 3.3V辅助输出
- J9: value OPTIONAL FPGA 3V3 IN -> 可选逻辑板3.3V输入
- JP1: value 1-2 ONBOARD / 2-3 FPGA -> 1-2板载 / 2-3逻辑板
Connections:
- net +3V3 renamed 本板3.3V
- net +3V3_ONBOARD renamed 保护后3.3V
- net +3V3_RAW renamed 板载3.3V
- net +3V3_SENS renamed 传感器3.3V
- net 传感器3.3V: no longer C112.1, C113.1, FB1.2
- net 3V3_FPGA_IN renamed 逻辑板3.3V_输入
- net BUCK_ENABLE renamed 使能
- net GND renamed 地
- net VLOGIC_IN renamed 降压输入
- new net 传感器电源: C112.1, C113.1, FB1.2
Other:
- note added: "JP1电源选择：只安装一个跳帽"
- note added: "传感器电源滤波 / 仅接已确认支持3.3V的成品模块"
- note added: "本板3.3V供给编码器、电流监测和安全逻辑；传感器信号接逻辑板。 裸芯片与成品模块的供电要求可能不同，须核对实际模块。"
- note added: "芯片标称2A能力不能代替接口与散热验收。 反馈取自保护开关前的稳压输出。 4.7µH位于手册允许的2.2-10µH范围内。"
- note added: "默认独立3.3V降压 / 初始负载预算0.5A"
- note added: "默认短接1-2：板载3.3V供电。 确认逻辑板电流余量后，才能改为2-3。 只能装一个跳帽，不能并联两个电源。 默认安装板载降压电路。"
- note removed: "2A IC capacity does not define connector/load budget. Feedback senses the buck output before protection. 4.7uH matches the allowed 2.2-10uH range."
- note removed: "DEFAULT: independent 3.3V buck / initial load budget 0.5A"
- note removed: "Default +3V3 powers encoders, current monitors and safety logic. Sensor signals connect to FPGA. Bare sensor chips and finished modules may need different supply levels; confirm actual modules."
- note removed: "Default shunt 1-2: onboard 3V3. 2-3 only after verifying FPGA headroom. Never fit two shunts. No hard paralleling. Onboard buck remains populated by default."
- note removed: "FILTERED SENSOR POWER / finished 3.3V-compatible modules only"
- note removed: "JP1: one shunt only / source selection"
- company: EdgeMind Robot -> EdgeMind机器人
- title: Independent 3V3 and source selector -> 独立3.3V与电源选择

Commit message: 10.3
Connections:
- net 传感器电源 is gone; now on net +3V3_SENS: C112.1, C113.1, FB1.2
- net 传感器3.3V renamed +3V3_SENS
- net 使能 renamed BUCK_ENABLE
- net 保护后3.3V renamed +3V3_ONBOARD
- net 地 renamed GND
- net 本板3.3V renamed +3V3
- net 板载3.3V renamed +3V3_RAW
- net 逻辑板3.3V_输入 renamed 3V3_FPGA_IN
- net 降压输入 renamed VLOGIC_IN
Changed lines of the file:
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@@
 		)
 	)
-	(global_label "传感器3.3V"
+	(global_label "+3V3_SENS"
 		(shape passive)
 		(at 175.26 234.95 180)
@@
 		)
 	)
-	(global_label "地"
+	(global_label "GND"
 		(shape passive)
 		(at 298.45 237.49 180)
@@
 		)
 	)
-	(global_label "传感器3.3V"
+	(global_label "+3V3_SENS"
 		(shape passive)
 		(at 298.45 185.42 180)
@@
 		)
 	)
-	(global_label "本板3.3V"
+	(global_label "+3V3"
 		(shape passive)
 		(at 44.45 179.07 180)
@@
 		)
 	)
-	(global_label "逻辑板3.3V_输入"
+	(global_label "3V3_FPGA_IN"
 		(shape passive)
 		(at 365.76 93.98 180)
@@
 		)
 	)
-	(global_label "传感器3.3V"
+	(global_label "+3V3_SENS"
 		(shape passive)
 		(at 298.45 234.95 180)
@@
 		)
 	)
-	(global_label "本板3.3V"
+	(global_label "+3V3"
 		(shape passive)
 		(at 93.98 238.76 180)
@@
 		)
 	)
-	(global_label "传感器3.3V"
+	(global_label "+3V3_SENS"
 		(shape passive)
 		(at 228.6 177.8 0)
@@
 		)
 	)
-	(global_label "本板3.3V"
+	(global_label "+3V3"
 		(shape passive)
 		(at 309.88 49.53 0)
@@
 		)
 	)
-	(global_label "传感器3.3V"
+	(global_label "+3V3_SENS"
 		(shape passive)
 		(at 351.79 177.8 0)
@@
 		)
 	)
-	(global_label "地"
+	(global_label "GND"
 		(shape passive)
 		(at 298.45 187.96 180)
@@
 		)
 	)
-	(global_label "传感器3.3V"
+	(global_label "+3V3_SENS"
 		(shape passive)
 		(at 175.26 185.42 180)
@@
 		)
 	)
-	(global_label "地"
+	(global_label "GND"
 		(shape passive)
 		(at 93.98 241.3 180)
@@
 		)
 	)
-	(global_label "地"
+	(global_label "GND"
 		(shape passive)
 		(at 175.26 237.49 180)
@@
 		)
 	)
-	(global_label "传感器3.3V"
+	(global_label "+3V3_SENS"
 		(shape passive)
 		(at 228.6 227.33 0)
@@
 		)
 	)
-	(global_label "地"
+	(global_label "GND"
 		(shape passive)
 		(at 175.26 187.96 180)
@@
 		)
 	)
-	(global_label "逻辑板3.3V_输入"
+	(global_label "3V3_FPGA_IN"
 		(shape passive)
 		(at 309.88 72.39 0)
@@
 		)
 	)
-	(global_label "地"
+	(global_label "GND"
 		(shape passive)
 		(at 365.76 96.52 180)
@@
 		)
 	)
-	(global_label "传感器3.3V"
+	(global_label "+3V3_SENS"
 		(shape passive)
 		(at 351.79 227.33 0)
@@
 		)
 	)
-	(global_label "逻辑板3.3V_输入"
+	(global_label "3V3_FPGA_IN"
 		(shape passive)
 		(at 284.48 52.07 180)
@@
 		)
 	)
-	(hierarchical_label "本板3.3V"
+	(hierarchical_label "+3V3"
 		(shape passive)
 		(at 284.48 49.53 180)
@@
 		)
 	)
-	(hierarchical_label "保护后3.3V"
+	(hierarchical_label "+3V3_ONBOARD"
 		(shape passive)
 		(at 284.48 46.99 180)
@@
 		)
 	)
-	(hierarchical_label "使能"
+	(hierarchical_label "BUCK_ENABLE"
 		(shape passive)
 		(at 76.2 69.85 180)
@@
 		)
 	)
-	(hierarchical_label "板载3.3V"
+	(hierarchical_label "+3V3_RAW"
 		(shape passive)
 		(at 207.01 64.77 0)
@@
 		)
 	)
-	(hierarchical_label "降压输入"
+	(hierarchical_label "VLOGIC_IN"
 		(shape passive)
 		(at 45.72 64.77 180)
@@
 		)
 	)
-	(hierarchical_label "传感器电源"
+	(hierarchical_label "+3V3_SENS"
 		(shape passive)
 		(at 111.76 179.07 0)
@@
 			)
 		)
-		(property "Value" "地"
+		(property "Value" "GND"
 			(at 228.6 176.53 0)
 			(hide yes)
@@
 			)
 		)
-		(property "Value" "地"
+		(property "Value" "GND"
 			(at 177.8 76.2 0)
 			(hide yes)
@@
 			)
 		)
-		(property "Value" "地"
+		(property "Value" "GND"
 			(at 105.41 185.42 0)
 			(hide yes)
@@
 			)
 		)
-		(property "Value" "地"
+		(property "Value" "GND"
 			(at 86.36 185.42 0)
 			(hide yes)
@@
 			)
 		)
-		(property "Value" "地"
+		(property "Value" "GND"
 			(at 351.79 176.53 0)
 			(hide yes)
@@
 			)
 		)
-		(property "Value" "地"
+		(property "Value" "GND"
 			(at 198.12 76.2 0)
 			(hide yes)
@@
 			)
 		)
-		(property "Value" "地"
+		(property "Value" "GND"
 			(at 351.79 226.06 0)
 			(hide yes)
@@
 			)
 		)
-		(property "Value" "地"
+		(property "Value" "GND"
 			(at 93.98 62.23 0)
 			(hide yes)
@@
 			)
 		)
-		(property "Value" "地"
+		(property "Value" "GND"
 			(at 228.6 226.06 0)
 			(hide yes)
@@
 			)
 		)
-		(property "Value" "地"
+		(property "Value" "GND"
 			(at 45.72 74.93 0)
 			(hide yes)

Commit message: 10.4
Other:
- moved on the sheet: C112, C113, C114, C115, C116, C117, FB1, J10, J11, J12, J13, J14
