File: pcb/power/kicad/04_motor_safety.kicad_sch (KiCad schematic)
At the start: 12 parts, among them J15 ESTOP NC LOOP, U10 74HC08D, U12 74HC74D, U13 MCP100-300DI/TO

Commit message: 10.3
Parts:
- J15: value ESTOP NC LOOP -> 急停常闭回路
Connections:
- net +3V3 renamed 本板3.3V
- net ESTOP_OK renamed 急停回路闭合
- net EXT_KILL_N renamed 外部故障
- net 外部故障: no longer U10.5
- net GND renamed 地
- net MOTOR_ARM renamed 电机解锁脉冲
- net 电机解锁脉冲: no longer R71.1
- net MOTOR_ARMED renamed 已解锁
- net 已解锁: no longer R73.1
- net MOTOR_PERMIT renamed 电机运行许可
- net 电机运行许可: no longer R70.1
- net MOTOR_POWER_OK renamed 动力正常
- net POR_OK renamed 上电复位完成
- new net 外部故障_低有效: U10.5
- new net 电机已解锁: R73.1
- new net 解锁脉冲: R71.1
- new net 运行许可: R70.1
Other:
- note added: "动力硬件锁存：上电关闭 / 常闭急停 / 解锁需要上升沿"
- note added: "急停断开、运行许可撤销、外部故障、欠压或过流均立即清除解锁。 条件恢复后还须发出解锁脉冲；逻辑板须在看门狗超时或堵转时撤销运行许可。 使用支持3.3V的74HC08与74HC74，不可换成74LS系列。"
- note removed: "MOTOR HARDWARE LATCH: power-on OFF / NC E-stop / explicit ARM rising edge"
- note removed: "Open E-stop / low PERMIT / external KILL / undervoltage / overcurrent clears immediately. Restore conditions then pulse ARM: no automatic restart. FPGA must drop PERMIT on watchdog/stall. HC08/HC74 are CMOS parts running at 3.3V. Do not substitute 74LS parts."
- company: EdgeMind Robot -> EdgeMind机器人
- title: E-stop and explicit arm latch -> 急停与显式解锁锁存

Commit message: 10.3
Connections:
- net 外部故障_低有效 is gone; now on net EXT_KILL_N: U10.5
- net 电机已解锁 is gone; now on net MOTOR_ARMED: R73.1
- net 解锁脉冲 is gone; now on net MOTOR_ARM: R71.1
- net 运行许可 is gone; now on net MOTOR_PERMIT: R70.1
- net 上电复位完成 renamed POR_OK
- net 动力正常 renamed MOTOR_POWER_OK
- net 地 renamed GND
- net 外部故障 renamed EXT_KILL_N
- net 已解锁 renamed MOTOR_ARMED
- net 急停回路闭合 renamed ESTOP_OK
- net 本板3.3V renamed +3V3
- net 电机解锁脉冲 renamed MOTOR_ARM
- net 电机运行许可 renamed MOTOR_PERMIT
Changed lines of the file:
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@@
 		)
 	)
-	(global_label "本板3.3V"
+	(global_label "+3V3"
 		(shape passive)
 		(at 73.66 226.06 0)
@@
 		)
 	)
-	(global_label "本板3.3V"
+	(global_label "+3V3"
 		(shape passive)
 		(at 53.34 207.01 0)
@@
 		)
 	)
-	(global_label "本板3.3V"
+	(global_label "+3V3"
 		(shape passive)
 		(at 137.16 226.06 0)
@@
 		)
 	)
-	(global_label "上电复位完成"
+	(global_label "POR_OK"
 		(shape passive)
 		(at 172.72 54.61 0)
@@
 		)
 	)
-	(global_label "电机运行许可"
+	(global_label "MOTOR_PERMIT"
 		(shape passive)
 		(at 228.6 66.04 180)
@@
 		)
 	)
-	(global_label "本板3.3V"
+	(global_label "+3V3"
 		(shape passive)
 		(at 116.84 209.55 0)
@@
 		)
 	)
-	(global_label "急停回路闭合"
+	(global_label "ESTOP_OK"
 		(shape passive)
 		(at 83.82 57.15 0)
@@
 		)
 	)
-	(global_label "上电复位完成"
+	(global_label "POR_OK"
 		(shape passive)
 		(at 228.6 101.6 180)
@@
 		)
 	)
-	(global_label "电机已解锁"
+	(global_label "MOTOR_ARMED"
 		(shape passive)
 		(at 369.57 212.09 0)
@@
 		)
 	)
-	(global_label "急停回路闭合"
+	(global_label "ESTOP_OK"
 		(shape passive)
 		(at 40.64 54.61 180)
@@
 		)
 	)
-	(global_label "本板3.3V"
+	(global_label "+3V3"
 		(shape passive)
 		(at 172.72 173.99 0)
@@
 		)
 	)
-	(global_label "本板3.3V"
+	(global_label "+3V3"
 		(shape passive)
 		(at 307.34 177.8 180)
@@
 		)
 	)
-	(global_label "本板3.3V"
+	(global_label "+3V3"
 		(shape passive)
 		(at 320.04 167.64 0)
@@
 		)
 	)
-	(global_label "本板3.3V"
+	(global_label "+3V3"
 		(shape passive)
 		(at 102.87 57.15 0)
@@
 		)
 	)
-	(global_label "本板3.3V"
+	(global_label "+3V3"
 		(shape passive)
 		(at 179.07 80.01 0)
@@
 		)
 	)
-	(global_label "外部故障_低有效"
+	(global_label "EXT_KILL_N"
 		(shape passive)
 		(at 228.6 106.68 180)
@@
 		)
 	)
-	(global_label "地"
+	(global_label "GND"
 		(shape passive)
 		(at 161.29 182.88 180)
@@
 		)
 	)
-	(global_label "急停回路闭合"
+	(global_label "ESTOP_OK"
 		(shape passive)
 		(at 228.6 60.96 180)
@@
 		)
 	)
-	(global_label "本板3.3V"
+	(global_label "+3V3"
 		(shape passive)
 		(at 154.94 40.64 0)
@@
 		)
 	)
-	(global_label "地"
+	(global_label "GND"
 		(shape passive)
 		(at 172.72 196.85 0)
@@
 		)
 	)
-	(global_label "电机解锁脉冲"
+	(global_label "MOTOR_ARM"
 		(shape passive)
 		(at 304.8 180.34 180)
@@
 		)
 	)
-	(global_label "地"
+	(global_label "GND"
 		(shape passive)
 		(at 161.29 185.42 180)
@@
 		)
 	)
-	(hierarchical_label "解锁脉冲"
+	(hierarchical_label "MOTOR_ARM"
 		(shape passive)
 		(at 71.12 86.36 0)
@@
 		)
 	)
-	(hierarchical_label "已解锁"
+	(hierarchical_label "MOTOR_ARMED"
 		(shape passive)
 		(at 335.28 177.8 0)
@@
 		)
 	)
-	(hierarchical_label "动力正常"
+	(hierarchical_label "MOTOR_POWER_OK"
 		(shape passive)
 		(at 228.6 147.32 180)
@@
 		)
 	)
-	(hierarchical_label "外部故障"
+	(hierarchical_label "EXT_KILL_N"
 		(shape passive)
 		(at 102.87 72.39 0)
@@
 		)
 	)
-	(hierarchical_label "运行许可"
+	(hierarchical_label "MOTOR_PERMIT"
 		(shape passive)
 		(at 40.64 86.36 0)
@@
 		)
 	)
-	(hierarchical_label "本板3.3V"
+	(hierarchical_label "+3V3"
 		(shape passive)
 		(at 40.64 52.07 180)
@@
 			)
 		)
-		(property "Value" "地"
+		(property "Value" "GND"
 			(at 154.94 52.07 0)
 			(hide yes)
@@
 			)
 		)
-		(property "Value" "地"
+		(property "Value" "GND"
 			(at 116.84 220.98 0)
 			(hide yes)
@@
 			)
 		)
-		(property "Value" "地"
+		(property "Value" "GND"
 			(at 137.16 224.79 0)
 			(hide yes)
@@
 			)
 		)
-		(property "Value" "地"
+		(property "Value" "GND"
 			(at 40.64 85.09 0)
 			(hide yes)
@@
 			)
 		)
-		(property "Value" "地"
+		(property "Value" "GND"
 			(at 369.57 210.82 0)
 			(hide yes)
@@
 			)
 		)
-		(property "Value" "地"
+		(property "Value" "GND"
 			(at 73.66 224.79 0)
 			(hide yes)
@@
 			)
 		)
-		(property "Value" "地"
+		(property "Value" "GND"
 			(at 71.12 85.09 0)
 			(hide yes)
@@
 			)
 		)
-		(property "Value" "地"
+		(property "Value" "GND"
 			(at 53.34 223.52 0)
 			(hide yes)
@@
 			)
 		)
-		(property "Value" "地"
+		(property "Value" "GND"
 			(at 83.82 55.88 0)
 			(hide yes)
@@
 			)
 		)
-		(property "Value" "地"
+		(property "Value" "GND"
 			(at 179.07 78.74 0)
 			(hide yes)

Commit message: 10.4
Other:
- moved on the sheet: C119, C120, R73, U10E, U12B, U12C
