File: pcb/power/kicad/08_rail_protection.kicad_sch (KiCad schematic)
At the start: 36 parts, among them Q10 AO4409, Q11 MMBT3904, Q12 AO3401A, Q13 MMBT3904, Q8 AO4409, Q9 MMBT3904, U27 LM393BIDR, U28 LM393BIDR, U29 LM393BIDR, U30 LM393BIDR

Commit message: 10.3
Connections:
- net +3V3 renamed 本板3.3V
- net +3V3_ONBOARD renamed 保护后3.3V
- net +3V3_RAW renamed 板载3.3V_稳压输出
- net 板载3.3V_稳压输出: no longer R114.1
- net +5V_AI renamed 计算板5V_稳压输出
- net 计算板5V_稳压输出: no longer R109.1
- net +5V_AI_OK renamed 计算板5V_电压正常
- net +5V_AI_PROT renamed 计算5V保护
- net +5V_FPGA renamed 逻辑板5V_稳压输出
- net 逻辑板5V_稳压输出: no longer R104.1
- net +5V_FPGA_OK renamed 逻辑板5V_电压正常
- net +5V_FPGA_PROT renamed 逻辑5V保护
- net 3V3_ONBOARD_OK renamed 板载3.3V_电压正常
- net BAT_WARN_N renamed 电池欠压告警_低有效
- net CURRENT_REF_1V217 renamed 过流基准_1.217V
- net GND renamed 地
- net MOTOR_POWER_OK renamed 电机供电正常
- net VBAT_SYS renamed 电池保护后母线
- net VM_L_IMON renamed 左电机_母线电流采样
- net VM_R_IMON renamed 右电机_母线电流采样
- net VREF_2V495 renamed 基准电压_2.495V
- new net 板载3.3V: R114.1
- new net 计算5V: R109.1
- new net 逻辑5V: R104.1
Other:
- note added: "5V过压关断 / 标称约5.364V / 计算板5V_保护输出"
- note added: "5V过压关断 / 标称约5.364V / 逻辑板5V_保护输出"
- note added: "分立过压关断方案用于控制成本；故障阶跃过冲和温升须实测。 本方案不保证所有状态下阻断反灌，接入板卡仍须核对电源选择与隔离。 母线过流阈值标称约3.04A；入口总保险板载，电池单体保护和模块限流仍须落实。"
- note added: "动力过流检测 / 滤波后母线电流 / 共用锁存清除"
- note added: "板载3.3V过压关断 / 标称约3.451V"
- note removed: "3V3 onboard OV cutoff ~3.451V"
- note removed: "5V OV cutoff ~5.364V / +5V_AI_PROT"
- note removed: "5V OV cutoff ~5.364V / +5V_FPGA_PROT"
- note removed: "Discrete OV disconnects are cost-oriented. Verify fault-step overshoot and thermal behavior. No claim of true reverse-current blocking: use supply selection/isolation on attached boards. Motor bus current threshold ~3.04A plus tolerance; fuse is harness protection, not winding limit."
- note removed: "MOTOR overcurrent / filtered bus current / common latch clear"
- company: EdgeMind Robot -> EdgeMind机器人
- title: Low-cost output OV disconnect -> 低成本输出过压关断
- moved on the sheet: R119, R120, R121, U29B

Commit message: 10.3
Connections:
- net 板载3.3V_稳压输出 is gone; now on net +3V3_RAW: Q12.2 (S), R116.2
- net 计算板5V_稳压输出 is gone; now on net +5V_AI: D8.1 (K), Q10.1 (S), Q10.2 (S), Q10.3 (S), R112.1
- net 逻辑板5V_稳压输出 is gone; now on net +5V_FPGA: D7.1 (K), Q8.1 (S), Q8.2 (S), Q8.3 (S), R107.1
- net 保护后3.3V renamed +3V3_ONBOARD
- net 右电机_母线电流采样 renamed VM_R_IMON
- net 地 renamed GND
- net 基准电压_2.495V renamed VREF_2V495
- net 左电机_母线电流采样 renamed VM_L_IMON
- net 本板3.3V renamed +3V3
- net 板载3.3V renamed +3V3_RAW
- net 板载3.3V_电压正常 renamed 3V3_ONBOARD_OK
- net 电机供电正常 renamed MOTOR_POWER_OK
- net 电池保护后母线 renamed VBAT_SYS
- net 电池欠压告警_低有效 renamed BAT_WARN_N
- net 计算5V renamed +5V_AI
- net 计算5V保护 renamed +5V_AI_PROT
- net 计算板5V_电压正常 renamed +5V_AI_OK
- net 过流基准_1.217V renamed CURRENT_REF_1V217
- net 逻辑5V renamed +5V_FPGA
- net 逻辑5V保护 renamed +5V_FPGA_PROT
- net 逻辑板5V_电压正常 renamed +5V_FPGA_OK
Other:
- note added: "计算板供电过压关断 / 标称约5.364V"
- note added: "逻辑板供电过压关断 / 标称约5.364V"
- note removed: "5V过压关断 / 标称约5.364V / 计算板5V_保护输出"
- note removed: "5V过压关断 / 标称约5.364V / 逻辑板5V_保护输出"
Changed lines of the file:
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@@
 		)
 	)
-	(text "5V过压关断 / 标称约5.364V / 逻辑板5V_保护输出"
+	(text "逻辑板供电过压关断 / 标称约5.364V"
 		(exclude_from_sim no)
 		(at 18 20 0)
@@
 		)
 	)
-	(text "5V过压关断 / 标称约5.364V / 计算板5V_保护输出"
+	(text "计算板供电过压关断 / 标称约5.364V"
 		(exclude_from_sim no)
 		(at 212.31 20 0)
@@
 		)
 	)
-	(global_label "计算板5V_稳压输出"
+	(global_label "+5V_AI"
 		(shape passive)
 		(at 364.49 27.94 0)
@@
 		)
 	)
-	(global_label "基准电压_2.495V"
+	(global_label "VREF_2V495"
 		(shape passive)
 		(at 63.5 58.42 180)
@@
 		)
 	)
-	(global_label "板载3.3V_电压正常"
+	(global_label "3V3_ONBOARD_OK"
 		(shape passive)
 		(at 88.9 246.38 0)
@@
 		)
 	)
-	(global_label "电池欠压告警_低有效"
+	(global_label "BAT_WARN_N"
 		(shape passive)
 		(at 293.37 179.07 0)
@@
 		)
 	)
-	(global_label "电池保护后母线"
+	(global_label "VBAT_SYS"
 		(shape passive)
 		(at 229.87 101.6 0)
@@
 		)
 	)
-	(global_label "电池保护后母线"
+	(global_label "VBAT_SYS"
 		(shape passive)
 		(at 121.92 97.79 0)
@@
 		)
 	)
-	(global_label "逻辑板5V_电压正常"
+	(global_label "+5V_FPGA_OK"
 		(shape passive)
 		(at 35.56 116.84 0)
@@
 		)
 	)
-	(global_label "地"
+	(global_label "GND"
 		(shape passive)
 		(at 67.31 105.41 180)
@@
 		)
 	)
-	(global_label "板载3.3V_稳压输出"
+	(global_label "+3V3_RAW"
 		(shape passive)
 		(at 149.86 170.18 180)
@@
 		)
 	)
-	(global_label "地"
+	(global_label "GND"
 		(shape passive)
 		(at 261.62 105.41 180)
@@
 		)
 	)
-	(global_label "过流基准_1.217V"
+	(global_label "CURRENT_REF_1V217"
 		(shape passive)
 		(at 266.7 213.36 180)
@@
 		)
 	)
-	(global_label "逻辑板5V_稳压输出"
+	(global_label "+5V_FPGA"
 		(shape passive)
 		(at 160.02 62.23 0)
@@
 		)
 	)
-	(global_label "电机供电正常"
+	(global_label "MOTOR_POWER_OK"
 		(shape passive)
 		(at 297.18 215.9 0)
@@
 		)
 	)
-	(global_label "电机供电正常"
+	(global_label "MOTOR_POWER_OK"
 		(shape passive)
 		(at 297.18 246.38 0)
@@
 		)
 	)
-	(global_label "电池保护后母线"
+	(global_label "VBAT_SYS"
 		(shape passive)
 		(at 35.56 101.6 0)
@@
 		)
 	)
-	(global_label "板载3.3V_稳压输出"
+	(global_label "+3V3_RAW"
 		(shape passive)
 		(at 160.02 198.12 0)
@@
 		)
 	)
-	(global_label "板载3.3V_电压正常"
+	(global_label "3V3_ONBOARD_OK"
 		(shape passive)
 		(at 93.98 184.15 0)
@@
 		)
 	)
-	(global_label "电池欠压告警_低有效"
+	(global_label "BAT_WARN_N"
 		(shape passive)
 		(at 353.06 181.61 0)
@@
 		)
 	)
-	(global_label "逻辑板5V_稳压输出"
+	(global_label "+5V_FPGA"
 		(shape passive)
 		(at 144.78 26.67 0)
@@
 		)
 	)
-	(global_label "计算板5V_稳压输出"
+	(global_label "+5V_AI"
 		(shape passive)
 		(at 339.09 26.67 0)
@@
 		)
 	)
-	(global_label "电池保护后母线"
+	(global_label "VBAT_SYS"
 		(shape passive)
 		(at 88.9 231.14 0)
@@
 		)
 	)
-	(global_label "基准电压_2.495V"
+	(global_label "VREF_2V495"
 		(shape passive)
 		(at 262.89 181.61 180)
@@
 		)
 	)
-	(global_label "基准电压_2.495V"
+	(global_label "VREF_2V495"
 		(shape passive)
 		(at 226.06 208.28 0)
@@
 		)
 	)
-	(global_label "过流基准_1.217V"
+	(global_label "CURRENT_REF_1V217"
 		(shape passive)
 		(at 226.06 228.6 0)
@@
 		)
 	)
-	(global_label "左电机_母线电流采样"
+	(global_label "VM_L_IMON"
 		(shape passive)
 		(at 266.7 218.44 180)
@@
 		)
 	)
-	(global_label "电池保护后母线"
+	(global_label "VBAT_SYS"
 		(shape passive)
 		(at 31.75 224.79 0)
@@
 		)
 	)
-	(global_label "右电机_母线电流采样"
+	(global_label "VM_R_IMON"
 		(shape passive)
 		(at 266.7 248.92 180)
@@
 		)
 	)
-	(global_label "基准电压_2.495V"
+	(global_label "VREF_2V495"
 		(shape passive)
 		(at 67.31 110.49 180)
@@
 		)
 	)
-	(global_label "基准电压_2.495V"
+	(global_label "VREF_2V495"
 		(shape passive)
 		(at 63.5 181.61 180)
@@
 		)
 	)
-	(global_label "逻辑板5V_电压正常"
+	(global_label "+5V_FPGA_OK"
 		(shape passive)
 		(at 93.98 60.96 0)
@@
 		)
 	)
-	(global_label "计算板5V_电压正常"
+	(global_label "+5V_AI_OK"
 		(shape passive)
 		(at 288.29 60.96 0)
@@
 		)
 	)
-	(global_label "电池保护后母线"
+	(global_label "VBAT_SYS"
 		(shape passive)
 		(at 316.23 97.79 0)
@@
 		)
 	)
-	(global_label "本板3.3V"
+	(global_label "+3V3"
 		(shape passive)
 		(at 353.06 166.37 0)
@@
 		)
 	)
-	(global_label "计算板5V_电压正常"
+	(global_label "+5V_AI_OK"
 		(shape passive)
 		(at 304.8 86.36 180)
@@
 		)
 	)
-	(global_label "逻辑板5V_电压正常"
+	(global_label "+5V_FPGA_OK"
 		(shape passive)
 		(at 110.49 86.36 180)
@@
 		)
 	)
-	(global_label "计算板5V_电压正常"
+	(global_label "+5V_AI_OK"
 		(shape passive)
 		(at 229.87 116.84 0)
@@
 		)
 	)
-	(global_label "计算板5V_稳压输出"
+	(global_label "+5V_AI"
 		(shape passive)
 		(at 354.33 62.23 0)
@@
 		)
 	)
-	(global_label "电池保护后母线"
+	(global_label "VBAT_SYS"
 		(shape passive)
 		(at 353.06 219.71 0)
@@
 		)
 	)
-	(global_label "电池保护后母线"
+	(global_label "VBAT_SYS"
 		(shape passive)
 		(at 240.03 156.21 0)
@@
 		)
 	)
-	(global_label "过流基准_1.217V"
+	(global_label "CURRENT_REF_1V217"
 		(shape passive)
 		(at 266.7 243.84 180)
@@
 		)
 	)
-	(global_label "基准电压_2.495V"
+	(global_label "VREF_2V495"
 		(shape passive)
 		(at 261.62 110.49 180)
@@
 		)
 	)
-	(global_label "逻辑板5V_稳压输出"
+	(global_label "+5V_FPGA"
 		(shape passive)
 		(at 170.18 27.94 0)
@@
 		)
 	)
-	(global_label "基准电压_2.495V"
+	(global_label "VREF_2V495"
 		(shape passive)
 		(at 257.81 58.42 180)
@@
 		)
 	)
-	(global_label "板载3.3V_电压正常"
+	(global_label "3V3_ONBOARD_OK"
 		(shape passive)
 		(at 102.87 219.71 180)
@@
 		)
 	)
-	(hierarchical_label "逻辑5V保护"
+	(hierarchical_label "+5V_FPGA_PROT"
 		(shape passive)
 		(at 190.5 45.72 0)
@@
 		)
 	)
-	(hierarchical_label "逻辑5V"
+	(hierarchical_label "+5V_FPGA"
 		(shape passive)
 		(at 40.64 43.18 0)
@@
 		)
 	)
-	(hierarchical_label "计算5V"
+	(hierarchical_label "+5V_AI"
 		(shape passive)
 		(at 234.95 43.18 0)
@@
 		)
 	)
-	(hierarchical_label "计算5V保护"
+	(hierarchical_label "+5V_AI_PROT"
 		(shape passive)
 		(at 384.81 45.72 0)
@@
 		)
 	)
-	(hierarchical_label "板载3.3V"
+	(hierarchical_label "+3V3_RAW"
 		(shape passive)
 		(at 40.64 166.37 0)
@@
 		)
 	)
-	(hierarchical_label "保护后3.3V"
+	(hierarchical_label "+3V3_ONBOARD"
 		(shape passive)
 		(at 170.18 170.18 0)
@@
 			)
 		)
-		(property "Value" "地"
+		(property "Value" "GND"
 			(at 52.07 237.49 0)
 			(hide yes)
@@
 			)
 		)
-		(property "Value" "地"
+		(property "Value" "GND"
 			(at 339.09 78.74 0)
 			(hide yes)
@@
 			)
 		)
-		(property "Value" "地"
+		(property "Value" "GND"
 			(at 40.64 190.5 0)
 			(hide yes)
@@
 			)
 		)
-		(property "Value" "地"
+		(property "Value" "GND"
 			(at 336.55 107.95 0)
 			(hide yes)
@@
 			)
 		)
-		(property "Value" "地"
+		(property "Value" "GND"
 			(at 234.95 67.31 0)
 			(hide yes)
@@
 			)
 		)
-		(property "Value" "地"
+		(property "Value" "GND"
 			(at 142.24 107.95 0)
 			(hide yes)
@@
 			)
 		)
-		(property "Value" "地"
+		(property "Value" "GND"
 			(at 240.03 180.34 0)
 			(hide yes)
@@
 			)
 		)
-		(property "Value" "地"
+		(property "Value" "GND"
 			(at 226.06 232.41 0)
 			(hide yes)
@@
 			)
 		)
-		(property "Value" "地"
+		(property "Value" "GND"
 			(at 142.24 212.09 0)
 			(hide yes)
@@
 			)
 		)
-		(property "Value" "地"
+		(property "Value" "GND"
 			(at 144.78 78.74 0)
 			(hide yes)
@@
 			)
 		)
-		(property "Value" "地"
+		(property "Value" "GND"
 			(at 40.64 67.31 0)
 			(hide yes)
@@
 			)
 		)
-		(property "Value" "地"
+		(property "Value" "GND"
 			(at 373.38 229.87 0)
 			(hide yes)

Commit message: 10.4
Other:
- moved on the sheet: C141, Q12, Q13, R114, R115, R116, R117, R118, U29A, U29C
