File: pcb/power/kicad/09_control_io.kicad_sch (KiCad schematic)
At the start: 6 parts, among them J1 LEFT CTRL, J18 POWER MONITOR / external ADC, J2 RIGHT CTRL

Commit message: 10.3
Parts:
- J1: value LEFT CTRL -> 左轮控制
- J18: value POWER MONITOR / external ADC -> 电源监测 / 外部模数转换
- J2: value RIGHT CTRL -> 右轮控制
Connections:
- net +3V3 renamed 本板3.3V
- net 3V3_FPGA_IN renamed 逻辑板3.3V_输入
- net BAT_ADC renamed 电池电压采样
- net BAT_WARN_N renamed 电池欠压告警_低有效
- net ENC_L_A_FPGA renamed 左编码器_A_逻辑板输入
- net ENC_L_B_FPGA renamed 左编码器_B_逻辑板输入
- net ENC_R_A_FPGA renamed 右编码器_A_逻辑板输入
- net ENC_R_B_FPGA renamed 右编码器_B_逻辑板输入
- net ESTOP_OK renamed 急停回路闭合
- net EXT_KILL_N renamed 外部故障
- net GND renamed 地
- net L_PWM_FWD_RAW renamed 左正转
- net L_PWM_REV_RAW renamed 左反转
- net MOTOR_ARM renamed 解锁脉冲
- net MOTOR_ARMED renamed 已解锁
- net 已解锁: no longer J18.8 (Pin_8)
- net MOTOR_PERMIT renamed 运行许可
- net MOTOR_POWER_OK renamed 电机供电正常
- net POR_OK renamed 上电复位完成
- net R_PWM_FWD_RAW renamed 右正转
- net R_PWM_REV_RAW renamed 右反转
- net USB1_FAULT_PULSE_N renamed 供电口1_故障脉冲_低有效
- net USB2_FAULT_PULSE_N renamed 供电口2_故障脉冲_低有效
- net VBAT_SYS renamed 电池保护后母线
- net VM_L_IMON renamed 左电机_母线电流采样
- net VM_R_IMON renamed 右电机_母线电流采样
- new net 电机已解锁: J18.8 (Pin_8)
Other:
- note added: "PCB封装与网络已同步，布局布线待完成。 仍须核对模块采样电阻、编码器版本与逻辑板供电接口。"
- note added: "控制接口 / 电源方向 / 互斥电源选择"
- note added: "电池采样：12.6V对应约2.71V，需要外部模数转换器。 J1第6脚与J2第3脚均为逻辑板3.3V输入， 默认与本板输出隔离，只接同一个电源域。 复位或看门狗超时时，运行许可必须为低。 安全检查后，以解锁脉冲的上升沿解锁。 外部故障脚接受开漏低电平。 荔枝派普通输入输出需要合适的电平转换。"
- note removed: "BAT_ADC: 12.6V -> 2.71V; requires external ADC. J1.6 and J2.3 = same FPGA 3V3 INPUT, not local 3V3 OUTPUT. JP1 isolates by default. Only connect one FPGA supply domain. PERMIT low during reset / watchdog timeout. ARM rising edge after safety checks. KILL_N accepts external open-drain fault. Lichee Pi GPIO needs appropriate level translation."
- note removed: "CONTROL / power direction / explicit source selection"
- note removed: "Do not fabricate the existing PCB using this schematic. Synchronization/layout is separate work. AT8236 Rsense / encoder variant / ACG720 Type-C supply path remain hardware verification items."
- company: EdgeMind Robot -> EdgeMind机器人
- title: FPGA control and monitor interfaces -> 逻辑板控制与电源监测接口

Commit message: 10.3
Connections:
- net 电机已解锁 is gone; now on net MOTOR_ARMED: J18.8 (Pin_8)
- net 上电复位完成 renamed POR_OK
- net 供电口1_故障脉冲_低有效 renamed USB1_FAULT_PULSE_N
- net 供电口2_故障脉冲_低有效 renamed USB2_FAULT_PULSE_N
- net 右反转 renamed R_PWM_REV_RAW
- net 右正转 renamed R_PWM_FWD_RAW
- net 右电机_母线电流采样 renamed VM_R_IMON
- net 右编码器_A_逻辑板输入 renamed ENC_R_A_FPGA
- net 右编码器_B_逻辑板输入 renamed ENC_R_B_FPGA
- net 地 renamed GND
- net 外部故障 renamed EXT_KILL_N
- net 左反转 renamed L_PWM_REV_RAW
- net 左正转 renamed L_PWM_FWD_RAW
- net 左电机_母线电流采样 renamed VM_L_IMON
- net 左编码器_A_逻辑板输入 renamed ENC_L_A_FPGA
- net 左编码器_B_逻辑板输入 renamed ENC_L_B_FPGA
- net 已解锁 renamed MOTOR_ARMED
- net 急停回路闭合 renamed ESTOP_OK
- net 本板3.3V renamed +3V3
- net 电机供电正常 renamed MOTOR_POWER_OK
- net 电池保护后母线 renamed VBAT_SYS
- net 电池欠压告警_低有效 renamed BAT_WARN_N
- net 电池电压采样 renamed BAT_ADC
- net 解锁脉冲 renamed MOTOR_ARM
- net 运行许可 renamed MOTOR_PERMIT
- net 逻辑板3.3V_输入 renamed 3V3_FPGA_IN
Changed lines of the file:
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@@
 		)
 	)
-	(global_label "地"
+	(global_label "GND"
 		(shape passive)
 		(at 149.86 162.56 180)
@@
 		)
 	)
-	(global_label "地"
+	(global_label "GND"
 		(shape passive)
 		(at 149.86 66.04 180)
@@
 		)
 	)
-	(global_label "供电口2_故障脉冲_低有效"
+	(global_label "USB2_FAULT_PULSE_N"
 		(shape passive)
 		(at 149.86 182.88 180)
@@
 		)
 	)
-	(global_label "供电口1_故障脉冲_低有效"
+	(global_label "USB1_FAULT_PULSE_N"
 		(shape passive)
 		(at 149.86 180.34 180)
@@
 		)
 	)
-	(global_label "急停回路闭合"
+	(global_label "ESTOP_OK"
 		(shape passive)
 		(at 149.86 185.42 180)
@@
 		)
 	)
-	(global_label "电池电压采样"
+	(global_label "BAT_ADC"
 		(shape passive)
 		(at 149.86 165.1 180)
@@
 		)
 	)
-	(global_label "逻辑板3.3V_输入"
+	(global_label "3V3_FPGA_IN"
 		(shape passive)
 		(at 335.28 60.96 180)
@@
 		)
 	)
-	(global_label "电池电压采样"
+	(global_label "BAT_ADC"
 		(shape passive)
 		(at 245.11 190.5 0)
@@
 		)
 	)
-	(global_label "地"
+	(global_label "GND"
 		(shape passive)
 		(at 335.28 63.5 180)
@@
 		)
 	)
-	(global_label "电机供电正常"
+	(global_label "MOTOR_POWER_OK"
 		(shape passive)
 		(at 149.86 175.26 180)
@@
 		)
 	)
-	(global_label "电池欠压告警_低有效"
+	(global_label "BAT_WARN_N"
 		(shape passive)
 		(at 149.86 167.64 180)
@@
 		)
 	)
-	(global_label "右电机_母线电流采样"
+	(global_label "VM_R_IMON"
 		(shape passive)
 		(at 149.86 172.72 180)
@@
 		)
 	)
-	(global_label "左编码器_A_逻辑板输入"
+	(global_label "ENC_L_A_FPGA"
 		(shape passive)
 		(at 149.86 71.12 180)
@@
 		)
 	)
-	(global_label "逻辑板3.3V_输入"
+	(global_label "3V3_FPGA_IN"
 		(shape passive)
 		(at 149.86 68.58 180)
@@
 		)
 	)
-	(global_label "左电机_母线电流采样"
+	(global_label "VM_L_IMON"
 		(shape passive)
 		(at 149.86 170.18 180)
@@
 		)
 	)
-	(global_label "右编码器_A_逻辑板输入"
+	(global_label "ENC_R_A_FPGA"
 		(shape passive)
 		(at 335.28 58.42 180)
@@
 		)
 	)
-	(global_label "左编码器_B_逻辑板输入"
+	(global_label "ENC_L_B_FPGA"
 		(shape passive)
 		(at 149.86 73.66 180)
@@
 		)
 	)
-	(global_label "电池保护后母线"
+	(global_label "VBAT_SYS"
 		(shape passive)
 		(at 245.11 170.18 0)
@@
 		)
 	)
-	(global_label "电机已解锁"
+	(global_label "MOTOR_ARMED"
 		(shape passive)
 		(at 149.86 177.8 180)
@@
 		)
 	)
-	(global_label "本板3.3V"
+	(global_label "+3V3"
 		(shape passive)
 		(at 149.86 160.02 180)
@@
 		)
 	)
-	(global_label "右编码器_B_逻辑板输入"
+	(global_label "ENC_R_B_FPGA"
 		(shape passive)
 		(at 335.28 55.88 180)
@@
 		)
 	)
-	(global_label "上电复位完成"
+	(global_label "POR_OK"
 		(shape passive)
 		(at 149.86 187.96 180)
@@
 		)
 	)
-	(hierarchical_label "左反转"
+	(hierarchical_label "L_PWM_REV_RAW"
 		(shape passive)
 		(at 149.86 58.42 180)
@@
 		)
 	)
-	(hierarchical_label "外部故障"
+	(hierarchical_label "EXT_KILL_N"
 		(shape passive)
 		(at 335.28 71.12 180)
@@
 		)
 	)
-	(hierarchical_label "运行许可"
+	(hierarchical_label "MOTOR_PERMIT"
 		(shape passive)
 		(at 149.86 63.5 180)
@@
 		)
 	)
-	(hierarchical_label "右正转"
+	(hierarchical_label "R_PWM_FWD_RAW"
 		(shape passive)
 		(at 335.28 66.04 180)
@@
 		)
 	)
-	(hierarchical_label "右反转"
+	(hierarchical_label "R_PWM_REV_RAW"
 		(shape passive)
 		(at 335.28 68.58 180)
@@
 		)
 	)
-	(hierarchical_label "解锁脉冲"
+	(hierarchical_label "MOTOR_ARM"
 		(shape passive)
 		(at 149.86 60.96 180)
@@
 		)
 	)
-	(hierarchical_label "左正转"
+	(hierarchical_label "L_PWM_FWD_RAW"
 		(shape passive)
 		(at 149.86 55.88 180)
@@
 		)
 	)
-	(hierarchical_label "已解锁"
+	(hierarchical_label "MOTOR_ARMED"
 		(shape passive)
 		(at 335.28 73.66 180)
@@
 			)
 		)
-		(property "Value" "地"
+		(property "Value" "GND"
 			(at 266.7 194.31 0)
 			(hide yes)
@@
 			)
 		)
-		(property "Value" "地"
+		(property "Value" "GND"
 			(at 245.11 194.31 0)
 			(hide yes)

Commit message: 10.4
Other:
- moved on the sheet: C143, J1, J18, J2, R124, R125
