File: pcb/power/kicad/ProPrj_power_2026-10-02.kicad_pcb (KiCad board)
At the start: 2 copper layers, 100 x 50 mm, 57 parts, among them CN1 XT60PW-M, J1 LAIL-PZ2.54-8P-L, J2 LAIL-PZ2.54-8P-L, J3 HX-XH2.54-6PZZ, J4 HX-XH2.54-6PZZ, J5 LAIL-PM2.54-7P-L, J6 LAIL-PM2.54-7P-L, J7 LAIL-PM2.54-7P-L, J8 LAIL-PM2.54-7P-L, SW2 SS-12D10L5, U1 MP2236GJ-Z, U5 MP2236GJ-Z

Commit message: 10.3
Parts:
- removed C61: 100nF, ProPrj_pow-easyedapro:C0805_C61
- removed H1, H2, H3, H4: MountingHole_3mm, ProPrj_pow-easyedapro:MountingHole_3mm
- removed J5, J6, J7, J8: LAIL-PM2.54-7P-L, ProPrj_pow-easyedapro:HDR-TH_LAIL-PM2.54-7P-L
- removed LED1: LED, ProPrj_pow-easyedapro:LED_0603
- removed R10, R14: 130K, ProPrj_pow-easyedapro:R0603
- removed R13, R7: 300K, ProPrj_pow-easyedapro:R0603
- removed R15: 10K, ProPrj_pow-easyedapro:R0603_R15
- removed R4: 10kΩ, ProPrj_pow-easyedapro:R0603_R4
- removed R5: 10kΩ, ProPrj_pow-easyedapro:R0603_R5
- removed R8: 10kΩ, ProPrj_pow-easyedapro:R0603_R8
- removed R9: 10kΩ, ProPrj_pow-easyedapro:R0603_R9
- removed SW2: SS-12D10L5, ProPrj_pow-easyedapro:SW-TH_SS-12D10L5
- added C101: 100uF/25V, Capacitor_THT:CP_Radial_D10.0mm_P5.00mm, F.Cu at (-49.8, 68.2)
- added C102: 100nF/50V, Capacitor_SMD:C_0805_2012Metric, F.Cu at (23.7, 78.4)
- added C103: 100nF/50V, Capacitor_SMD:C_0805_2012Metric, F.Cu at (23.7, 81.4)
- added C104: 1uF/25V, Capacitor_SMD:C_0805_2012Metric, F.Cu at (258.0, 107.2)
- added C105: 4.7uF/10V, Capacitor_SMD:C_0805_2012Metric, F.Cu at (258.0, 104.2)
- added C106: 1uF/25V, Capacitor_SMD:C_0805_2012Metric, F.Cu at (223.9, 103.2)
- added C107: 4.7uF/10V, Capacitor_SMD:C_0805_2012Metric, F.Cu at (223.9, 100.2)
- added C108: 10uF/25V, Capacitor_SMD:C_0805_2012Metric, F.Cu at (98.9, 151.4)
- added C109: 100nF/50V, Capacitor_SMD:C_0603_1608Metric, F.Cu at (90.7, 177.4)
- added C110: 22uF/10V, Capacitor_SMD:C_0805_2012Metric, F.Cu at (98.9, 154.4)
- added C111: 22uF/10V, Capacitor_SMD:C_0805_2012Metric, F.Cu at (98.9, 157.4)
- added C112: 10uF/10V, Capacitor_SMD:C_0805_2012Metric, F.Cu at (103.3, 151.4)
- added C113: 100nF/50V, Capacitor_SMD:C_0805_2012Metric, F.Cu at (103.3, 154.4)
- added C114: 100nF/50V, Capacitor_SMD:C_0805_2012Metric, F.Cu at (103.3, 157.4)
- added C115: 100nF/50V, Capacitor_SMD:C_0805_2012Metric, F.Cu at (107.8, 151.4)
- added C116: 100nF/50V, Capacitor_SMD:C_0805_2012Metric, F.Cu at (107.8, 154.4)
- added C117: 100nF/50V, Capacitor_SMD:C_0805_2012Metric, F.Cu at (107.8, 157.4)
- added C118: 100nF/50V, Capacitor_SMD:C_0805_2012Metric, F.Cu at (68.6, 165.9)
- added C119: 100nF/50V, Capacitor_SMD:C_0805_2012Metric, F.Cu at (68.6, 169.0)
- added C120: 100nF/50V, Capacitor_SMD:C_0805_2012Metric, F.Cu at (68.6, 172.0)
- added C121: 100nF/50V, Capacitor_SMD:C_0805_2012Metric, F.Cu at (161.6, 155.1)
- added C122: 470uF/25V, Capacitor_THT:CP_Radial_D10.0mm_P5.00mm, F.Cu at (135.6, 21.0)
- added C123: 100nF/50V, Capacitor_SMD:C_0805_2012Metric, F.Cu at (137.8, 29.5)
- added C124: 100nF/50V, Capacitor_SMD:C_0805_2012Metric, F.Cu at (137.8, 32.5)
- added C125: 1uF/25V, Capacitor_SMD:C_0603_1608Metric, F.Cu at (132.8, 29.5)
- added C126: 1uF/25V, Capacitor_SMD:C_0603_1608Metric, F.Cu at (-13.3, 176.6)
- added C127: 100nF/50V, Capacitor_SMD:C_0805_2012Metric, F.Cu at (-1.02, 180.4)
- added C128: 1nF/C0G, Capacitor_SMD:C_0603_1608Metric, F.Cu at (-13.3, 179.2)
- added C129: 1nF/C0G, Capacitor_SMD:C_0603_1608Metric, F.Cu at (-13.3, 181.7)
- added C130: 100nF/50V, Capacitor_SMD:C_0805_2012Metric, F.Cu at (-1.02, 183.4)
- added C131: 470uF/25V, Capacitor_THT:CP_Radial_D10.0mm_P5.00mm, F.Cu at (116.5, 53.2)
- added C132: 100nF/50V, Capacitor_SMD:C_0805_2012Metric, F.Cu at (127.0, 60.1)
- added C133: 100nF/50V, Capacitor_SMD:C_0805_2012Metric, F.Cu at (127.0, 63.1)
- added C134: 1uF/25V, Capacitor_SMD:C_0603_1608Metric, F.Cu at (128.7, 45.4)
- added C135: 1uF/25V, Capacitor_SMD:C_0603_1608Metric, F.Cu at (29.2, 215.7)
- added C136: 1nF/C0G, Capacitor_SMD:C_0603_1608Metric, F.Cu at (29.2, 218.2)
- added C137: 1nF/C0G, Capacitor_SMD:C_0603_1608Metric, F.Cu at (29.2, 220.8)
- added C138: 100nF/50V, Capacitor_SMD:C_0805_2012Metric, F.Cu at (13.5, 250.5)
- added C139: 100nF/50V, Capacitor_SMD:C_0805_2012Metric, F.Cu at (241.8, 25.9)
- added C140: 100nF/50V, Capacitor_SMD:C_0805_2012Metric, F.Cu at (238.9, 56.3)
- added C141: 100nF/50V, Capacitor_SMD:C_0805_2012Metric, F.Cu at (271.1, 21.8)
- added C142: 100nF/50V, Capacitor_SMD:C_0805_2012Metric, F.Cu at (271.8, 58.9)
- added C143: 100nF/25V, Capacitor_SMD:C_0603_1608Metric, F.Cu at (179.5, 119.4)
- added D2: BZT52C12, Diode_SMD:D_SOD-123, F.Cu at (-22.5, 26.1)
- added D3: BZT52C12, Diode_SMD:D_SOD-123, F.Cu at (-31.6, 69.2)
- added D4: BZT52C12, Diode_SMD:D_SOD-123, F.Cu at (158.8, 168.7)
- added D5: BZT52C12, Diode_SMD:D_SOD-123, F.Cu at (158.8, 172.0)
- added D6: BZT52C12, Diode_SMD:D_SOD-123, F.Cu at (158.8, 175.4)
- added D7: BZT52C12, Diode_SMD:D_SOD-123, F.Cu at (247.0, 26.0)
- added D8: BZT52C12, Diode_SMD:D_SOD-123, F.Cu at (244.0, 56.8)
- added F1: 10A/32V MINI总保险, Fuse:Fuseholder_Blade_Mini_Keystone_3568, F.Cu at (-18.9, 35.2)
- added FB1: 220Ω@100MHz / 1A, Inductor_SMD:L_0805_2012Metric, F.Cu at (112.3, 155.9)
- added J10: 惯性传感器电源, Connector_JST:JST_PH_B2B-PH-K_1x02_P2.00mm_Vertical, F.Cu at (91.7, 152.6)
- added J11: 测距传感器1电源, Connector_JST:JST_PH_B2B-PH-K_1x02_P2.00mm_Vertical, F.Cu at (91.7, 159.2)
- added J12: 测距传感器2电源, Connector_JST:JST_PH_B2B-PH-K_1x02_P2.00mm_Vertical, F.Cu at (91.7, 165.7)
- added J13: 测距传感器3电源, Connector_JST:JST_PH_B2B-PH-K_1x02_P2.00mm_Vertical, F.Cu at (91.7, 172.3)
- added J14: 3.3V辅助输出, TerminalBlock_Phoenix:TerminalBlock_Phoenix_MKDS-1,5-2-5.08_1x02_P5.08mm_Horizontal, F.Cu at (100.2, 165.2)
- added J15: 急停常闭回路, TerminalBlock_Phoenix:TerminalBlock_Phoenix_MKDS-1,5-2-5.08_1x02_P5.08mm_Horizontal, F.Cu at (57.7, 170.7)
- added J16: 左回生泄放 / 外接3.3Ω, TerminalBlock_Phoenix:TerminalBlock_Phoenix_MKDS-1,5-2-5.08_1x02_P5.08mm_Horizontal, F.Cu at (139.2, 155.4)
- added J17: 右回生泄放 / 外接3.3Ω, TerminalBlock_Phoenix:TerminalBlock_Phoenix_MKDS-1,5-2-5.08_1x02_P5.08mm_Horizontal, F.Cu at (139.2, 167.5)
- added J18: 电源监测 / 外部模数转换, Connector_PinHeader_2.54mm:PinHeader_1x12_P2.54mm_Vertical, F.Cu at (175.2, 98.0)
- added J9: 可选逻辑板3.3V输入, Connector_PinHeader_2.54mm:PinHeader_1x02_P2.54mm_Vertical, F.Cu at (108.9, 173.4)
- added JP1: 1-2板载 / 2-3逻辑板, Connector_PinHeader_2.54mm:PinHeader_1x03_P2.54mm_Vertical, F.Cu at (111.2, 161.2)
- added L3: 4.7uH, Inductor_SMD:L_Changjiang_FXL0630, F.Cu at (101.6, 175.1)
- added Q1: IRF4905, Package_TO_SOT_THT:TO-220-3_Vertical, F.Cu at (-51.6, 38.2)
- added Q10: AO4409, Package_SO:SOIC-8_3.9x4.9mm_P1.27mm, F.Cu at (227.5, 61.8)
- added Q11: MMBT3904, Package_TO_SOT_SMD:SOT-23, F.Cu at (234.2, 58.5)
- added Q12: AO3401A, Package_TO_SOT_SMD:SOT-23, F.Cu at (266.4, 25.4)
- added Q13: MMBT3904, Package_TO_SOT_SMD:SOT-23, F.Cu at (266.4, 29.9)
- added Q2: IRF4905, Package_TO_SOT_THT:TO-220-3_Vertical, F.Cu at (151.1, 153.1)
- added Q3: IRF4905, Package_TO_SOT_THT:TO-220-3_Vertical, F.Cu at (-51.9, 81.3)
- added Q4: MMBT3904, Package_TO_SOT_SMD:SOT-23, F.Cu at (-24.4, 79.3)
- added Q5: MMBT3904, Package_TO_SOT_SMD:SOT-23, F.Cu at (161.8, 151.4)
- added Q6: IRLZ44N, Package_TO_SOT_THT:TO-220-3_Vertical, F.Cu at (151.1, 159.0)
- added Q7: IRLZ44N, Package_TO_SOT_THT:TO-220-3_Vertical, F.Cu at (151.1, 165.0)
- added Q8: AO4409, Package_SO:SOIC-8_3.9x4.9mm_P1.27mm, F.Cu at (230.5, 27.7)
- added Q9: MMBT3904, Package_TO_SOT_SMD:SOT-23, F.Cu at (237.2, 26.6)
- added R100: 100R, Resistor_SMD:R_0603_1608Metric, F.Cu at (33.2, 223.3)
- added R101: 10k, Resistor_SMD:R_0603_1608Metric, F.Cu at (37.2, 213.2)
- added R102: 100R, Resistor_SMD:R_0603_1608Metric, F.Cu at (37.2, 215.7)
- added R103: 10k, Resistor_SMD:R_0603_1608Metric, F.Cu at (37.2, 218.2)
- added R104: 11.5k/0.1%, Resistor_SMD:R_0603_1608Metric, F.Cu at (244.0, 34.4)
- added R105: 10.0k/0.1%, Resistor_SMD:R_0603_1608Metric, F.Cu at (244.0, 36.9)
- added R106: 10k, Resistor_SMD:R_0603_1608Metric, F.Cu at (244.0, 39.4)
- added R107: 1k, Resistor_SMD:R_0603_1608Metric, F.Cu at (244.0, 41.9)
- added R108: 4.7k, Resistor_SMD:R_0603_1608Metric, F.Cu at (244.0, 44.4)
- added R109: 11.5k/0.1%, Resistor_SMD:R_0603_1608Metric, F.Cu at (237.7, 70.9)
- added R110: 10.0k/0.1%, Resistor_SMD:R_0603_1608Metric, F.Cu at (237.7, 73.4)
- added R111: 10k, Resistor_SMD:R_0603_1608Metric, F.Cu at (237.7, 75.9)
- added R112: 1k, Resistor_SMD:R_0603_1608Metric, F.Cu at (237.7, 78.4)
- added R113: 4.7k, Resistor_SMD:R_0603_1608Metric, F.Cu at (237.7, 80.9)
- added R114: 3.83k/0.1%, Resistor_SMD:R_0603_1608Metric, F.Cu at (274.0, 33.4)
- added R115: 10.0k/0.1%, Resistor_SMD:R_0603_1608Metric, F.Cu at (274.0, 35.9)
- added R116: 1k, Resistor_SMD:R_0603_1608Metric, F.Cu at (274.0, 38.4)
- added R117: 4.7k, Resistor_SMD:R_0603_1608Metric, F.Cu at (274.0, 40.9)
- added R118: 10k, Resistor_SMD:R_0603_1608Metric, F.Cu at (274.0, 43.4)
- added R119: 30.9k/0.1%, Resistor_SMD:R_0603_1608Metric, F.Cu at (278.7, 67.5)
- added R120: 10.0k/0.1%, Resistor_SMD:R_0603_1608Metric, F.Cu at (278.7, 70.0)
- added R121: 10k, Resistor_SMD:R_0603_1608Metric, F.Cu at (278.7, 72.5)
- added R122: 10.5k/0.1%, Resistor_SMD:R_0603_1608Metric, F.Cu at (278.7, 75.0)
- added R123: 10.0k/0.1%, Resistor_SMD:R_0603_1608Metric, F.Cu at (278.7, 77.5)
- added R124: 100k/0.1%, Resistor_SMD:R_0603_1608Metric, F.Cu at (179.5, 121.9)
- added R125: 27.4k/0.1%, Resistor_SMD:R_0603_1608Metric, F.Cu at (179.5, 124.4)
- added R51: 100k, Resistor_SMD:R_0603_1608Metric, F.Cu at (-41.0, 41.2)
- added R52: 2.2k, Resistor_SMD:R_0603_1608Metric, F.Cu at (-41.3, 80.9)
- added R53: 10k, Resistor_SMD:R_0603_1608Metric, F.Cu at (-41.3, 83.4)
- added R54: 4.7k, Resistor_SMD:R_0603_1608Metric, F.Cu at (-41.3, 85.9)
- added R55: 26.1k/0.1%, Resistor_SMD:R_0603_1608Metric, F.Cu at (11.4, 82.2)
- added R56: 10.0k/0.1%, Resistor_SMD:R_0603_1608Metric, F.Cu at (15.4, 72.2)
- added R57: 46.4k/0.1%, Resistor_SMD:R_0603_1608Metric, F.Cu at (15.4, 74.7)
- added R58: 10.0k/0.1%, Resistor_SMD:R_0603_1608Metric, F.Cu at (15.4, 77.2)
- added R59: 10k, Resistor_SMD:R_0603_1608Metric, F.Cu at (15.4, 79.7)
- added R60: 28.7k/0.1%, Resistor_SMD:R_0603_1608Metric, F.Cu at (15.4, 82.2)
- added R61: 10.0k/0.1%, Resistor_SMD:R_0603_1608Metric, F.Cu at (19.4, 72.2)
- added R62: 46.4k/0.1%, Resistor_SMD:R_0603_1608Metric, F.Cu at (19.4, 74.7)
- added R63: 10.0k/0.1%, Resistor_SMD:R_0603_1608Metric, F.Cu at (19.4, 77.2)
- added R64: 10k, Resistor_SMD:R_0603_1608Metric, F.Cu at (19.4, 79.7)
- added R65: 150k/1%, Resistor_SMD:R_0603_1608Metric, F.Cu at (278.7, 107.0)
- added R66: 10k, Resistor_SMD:R_0603_1608Metric, F.Cu at (278.7, 104.5)
- added R67: 150k/1%, Resistor_SMD:R_0603_1608Metric, F.Cu at (242.7, 110.2)
- added R68: 10k, Resistor_SMD:R_0603_1608Metric, F.Cu at (242.7, 107.7)
- added R69: 10k, Resistor_SMD:R_0603_1608Metric, F.Cu at (52.1, 165.7)
- added R70: 10k, Resistor_SMD:R_0603_1608Metric, F.Cu at (52.1, 168.2)
- added R71: 10k, Resistor_SMD:R_0603_1608Metric, F.Cu at (52.1, 170.7)
- added R72: 10k, Resistor_SMD:R_0603_1608Metric, F.Cu at (52.1, 173.2)
- added R73: 4.7k, Resistor_SMD:R_0603_1608Metric, F.Cu at (52.1, 175.7)
- added R74: 10k, Resistor_SMD:R_0603_1608Metric, F.Cu at (149.8, 168.2)
- added R75: 4.7k, Resistor_SMD:R_0603_1608Metric, F.Cu at (149.8, 170.8)
- added R76: 51.1k/0.1%, Resistor_SMD:R_0603_1608Metric, F.Cu at (149.8, 173.3)
- added R77: 10.0k/0.1%, Resistor_SMD:R_0603_1608Metric, F.Cu at (149.8, 175.8)
- added R78: 4.7k, Resistor_SMD:R_0603_1608Metric, F.Cu at (149.8, 178.3)
- added R79: 1M, Resistor_SMD:R_0603_1608Metric, F.Cu at (153.8, 168.2)
- added R80: 51.1k/0.1%, Resistor_SMD:R_0603_1608Metric, F.Cu at (153.8, 170.8)
- added R81: 10.0k/0.1%, Resistor_SMD:R_0603_1608Metric, F.Cu at (153.8, 173.3)
- added R82: 4.7k, Resistor_SMD:R_0603_1608Metric, F.Cu at (153.8, 175.8)
- added R83: 1M, Resistor_SMD:R_0603_1608Metric, F.Cu at (153.8, 178.3)
- added R84: 0.020R/1%/1W, Resistor_SMD:R_2512_6332Metric, F.Cu at (118.7, 32.3)
- added R85: 1k, Resistor_SMD:R_0603_1608Metric, F.Cu at (132.8, 34.0)
- added R86: 1k, Resistor_SMD:R_0603_1608Metric, F.Cu at (-9.26, 174.1)
- added R87: 100k, Resistor_SMD:R_0603_1608Metric, F.Cu at (-9.26, 176.6)
- added R88: 10k, Resistor_SMD:R_0603_1608Metric, F.Cu at (-9.26, 179.2)
- added R89: 10k, Resistor_SMD:R_0603_1608Metric, F.Cu at (-9.26, 181.7)
- added R90: 100R, Resistor_SMD:R_0603_1608Metric, F.Cu at (-9.26, 184.2)
- added R91: 10k, Resistor_SMD:R_0603_1608Metric, F.Cu at (-5.25, 174.1)
- added R92: 100R, Resistor_SMD:R_0603_1608Metric, F.Cu at (-5.25, 176.6)
- added R93: 10k, Resistor_SMD:R_0603_1608Metric, F.Cu at (-5.25, 179.2)
- added R94: 0.020R/1%/1W, Resistor_SMD:R_2512_6332Metric, F.Cu at (131.6, 52.8)
- added R95: 1k, Resistor_SMD:R_0603_1608Metric, F.Cu at (129.3, 49.0)
- added R96: 1k, Resistor_SMD:R_0603_1608Metric, F.Cu at (33.2, 213.2)
- added R97: 100k, Resistor_SMD:R_0603_1608Metric, F.Cu at (33.2, 215.7)
- added R98: 10k, Resistor_SMD:R_0603_1608Metric, F.Cu at (33.2, 218.2)
- added R99: 10k, Resistor_SMD:R_0603_1608Metric, F.Cu at (33.2, 220.8)
- added RV1: 10k/3296W, Potentiometer_THT:Potentiometer_Bourns_3296W_Vertical, F.Cu at (0.95, 156.6)
- added RV2: 10k/3296W, Potentiometer_THT:Potentiometer_Bourns_3296W_Vertical, F.Cu at (7.54, 246.5)
- added TP1: 电机总开关输出, TestPoint:TestPoint_Pad_D2.0mm, F.Cu at (161.4, 158.6)
- added U10: 74HC08D, Package_SO:SOIC-14_3.9x8.7mm_P1.27mm, F.Cu at (54.4, 159.3)
- added U11: 74HC08D, Package_SO:SOIC-14_3.9x8.7mm_P1.27mm, F.Cu at (-19.8, 211.8)
- added U12: 74HC74D, Package_SO:SOIC-14_3.9x8.7mm_P1.27mm, F.Cu at (62.8, 159.3)
- added U13: MCP100-300DI/TO, Package_TO_SOT_THT:TO-92_Inline, F.Cu at (69.0, 157.3)
- added U2: AT8236双路模块, EdgeMind_Module:AT8236_Dual_PinSocket_2x7_P2.54_Row23.0005mm, F.Cu at (-45.0, 133.0)
- added U21: TL431BIDBZR, Package_TO_SOT_SMD:SOT-23, F.Cu at (-24.4, 83.8)
- added U22: LM393BIDR, Package_SO:SOIC-8_3.9x4.9mm_P1.27mm, F.Cu at (24.0, 56.5)
- added U23: LM393BIDR, Package_SO:SOIC-8_3.9x4.9mm_P1.27mm, F.Cu at (24.0, 63.1)
- added U24: LM393BIDR, Package_SO:SOIC-8_3.9x4.9mm_P1.27mm, F.Cu at (139.8, 176.8)
- added U25: INA180A1IDBVR, Package_TO_SOT_SMD:SOT-23-5, F.Cu at (125.6, 32.2)
- added U26: INA180A1IDBVR, Package_TO_SOT_SMD:SOT-23-5, F.Cu at (136.3, 60.2)
- added U27: LM393BIDR, Package_SO:SOIC-8_3.9x4.9mm_P1.27mm, F.Cu at (230.5, 40.9)
- added U28: LM393BIDR, Package_SO:SOIC-8_3.9x4.9mm_P1.27mm, F.Cu at (227.5, 74.9)
- added U29: LM393BIDR, Package_SO:SOIC-8_3.9x4.9mm_P1.27mm, F.Cu at (265.0, 38.5)
- added U3: AP63203WU-7, Package_TO_SOT_SMD:TSOT-23-6, F.Cu at (112.6, 152.3)
- added U30: LM393BIDR, Package_SO:SOIC-8_3.9x4.9mm_P1.27mm, F.Cu at (265.1, 75.6)
- added U4: AT8236双路模块, EdgeMind_Module:AT8236_Dual_PinSocket_2x7_P2.54_Row23.1275mm, F.Cu at (1.75, 214.3)
- added U7: HUSB305-02, Package_TO_SOT_SMD:TSOT-23-8, F.Cu at (266.9, 111.8)
- added U8: HUSB305-02, Package_TO_SOT_SMD:TSOT-23-8, F.Cu at (233.9, 110.1)
- C1, C10, C12, C13, C2, C3, C4, C5, C8, C9: value 22uF -> 22uF/25V; footprint ProPrj_pow-easyedapro:C0805 -> Capacitor_SMD:C_0805_2012Metric
- C11, C16: value 1uf -> 1uF/25V; footprint ProPrj_pow-easyedapro:C0603 -> Capacitor_SMD:C_0805_2012Metric
- C14, C6: value 100nF -> 100nF/50V; footprint ProPrj_pow-easyedapro:C0603 -> Capacitor_SMD:C_0603_1608Metric
- C15, C7: value 220PF -> 220pF/C0G; footprint ProPrj_pow-easyedapro:C0603 -> Capacitor_SMD:C_0603_1608Metric
- C58: value 100uF -> 470uF/35V; footprint ProPrj_pow-easyedapro:C0805_C58 -> Capacitor_THT:CP_Radial_D10.0mm_P5.00mm
- C59: value 10uF -> 10uF/50V; footprint ProPrj_pow-easyedapro:C0805_C59 -> Capacitor_SMD:C_0805_2012Metric
- C60: value 100nF -> 100nF/50V; footprint ProPrj_pow-easyedapro:C0805_C60 -> Capacitor_SMD:C_0805_2012Metric
- CN1: value XT60PW-M -> XT60PW-M / 三串电池; footprint ProPrj_pow-easyedapro:CONN-TH_XT60PW-M -> Connector_AMASS:AMASS_XT60PW-M_1x02_P7.20mm_Horizontal
- D1: value SMF12A -> SMBJ15CA; footprint ProPrj_pow-easyedapro:SOD-123_L2.7-W1.8-LS3.7-RD -> Diode_SMD:D_SMB
- J1: value LAIL-PZ2.54-8P-L -> 左轮控制; footprint ProPrj_pow-easyedapro:CONN-TH_LAIL-PZ2.54-8P-L -> Connector_PinHeader_2.54mm:PinHeader_1x08_P2.54mm_Vertical
- J2: value LAIL-PZ2.54-8P-L -> 右轮控制; footprint ProPrj_pow-easyedapro:CONN-TH_LAIL-PZ2.54-8P-L -> Connector_PinHeader_2.54mm:PinHeader_1x08_P2.54mm_Vertical
- J3, J4: value HX-XH2.54-6PZZ -> MG513电机 / 核对线序; footprint ProPrj_pow-easyedapro:CONN-TH_6P-P2.50_BX-XH2.54-6PZZ -> Connector_JST:JST_XH_B6B-XH-A_1x06_P2.50mm_Vertical
- L1, L2: value 4.8uh -> 4.7uH; footprint ProPrj_pow-easyedapro:IND-SMD_L7.3-W6.6 -> Inductor_SMD:L_Changjiang_FXL0630
- R1, R6: footprint ProPrj_pow-easyedapro:R0603 -> Resistor_SMD:R_0603_1608Metric
- R11, R2: value 82K -> 82.5k/0.1%; footprint ProPrj_pow-easyedapro:R0603 -> Resistor_SMD:R_0603_1608Metric
- R12, R3: value 11.1K -> 11.0k/0.1%; footprint ProPrj_pow-easyedapro:R0603 -> Resistor_SMD:R_0603_1608Metric
- U1, U5: footprint ProPrj_pow-easyedapro:TSOT-23-8_L2.9-W1.6-P0.65-LS2.8-BL -> Package_TO_SOT_SMD:TSOT-23-8
- USB1, USB2: value LAIL-TYPE-C-16PIN-08-WT -> USB4125-GF-A / 六针供电; footprint ProPrj_pow-easyedapro:TYPE-C-SMD_LAIL-TYPE-C-16PIN-08-WT -> Connector_USB:USB_C_Receptacle_GCT_USB4125-xx-x_6P_TopMnt_Horizontal
- moved J4 198.2 mm to (19.2, 246.3)
- moved J3 196.1 mm to (-31.2, 176.2)
- moved C58 185.5 mm to (-51.2, 17.0), turned to 0 degrees
- moved D1 184.7 mm to (-50.6, 49.0)
- moved CN1 168.4 mm to (-37.9, 8.40), turned to 0 degrees
- moved C60 158.6 mm to (-28.7, 44.5), turned to 0 degrees
- moved C59 157.6 mm to (-28.7, 41.5), turned to 0 degrees
- moved C8 153.6 mm to (273.9, 122.5), turned to 0 degrees
- moved R6 152.4 mm to (283.2, 136.3), turned to 0 degrees
- moved R12 151.9 mm to (283.2, 141.3), turned to 0 degrees
- moved C10 151.8 mm to (273.9, 128.5), turned to 0 degrees
- moved C9 149.3 mm to (273.9, 125.5), turned to 0 degrees
- moved R11 149.2 mm to (283.2, 138.8), turned to 0 degrees
- moved C14 148.8 mm to (279.2, 136.3), turned to 0 degrees
- moved C15 142.8 mm to (279.2, 138.8), turned to 0 degrees
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Connections:
- C1 pad 1: GND -> 降压电源输入
- C1 pad 2: VCCIN -> 地
- C10 pad 1: GND -> 降压电源输入
- C10 pad 2: VCCIN -> 地
- C11 pad 2: GND -> 地
- C12 pad 1: VCCOUT1 -> 计算板5V_稳压输出
- C12 pad 2: GND -> 地
- C13 pad 1: VCCOUT1 -> 计算板5V_稳压输出
- C13 pad 2: GND -> 地
- C15 pad 1: VCCOUT1 -> 计算板5V_稳压输出
- C16 pad 2: GND -> 地
- C2 pad 1: GND -> 降压电源输入
- C2 pad 2: VCCIN -> 地
- C3 pad 1: GND -> 降压电源输入
- C3 pad 2: VCCIN -> 地
- C4 pad 1: VCCOUT -> 逻辑板5V_稳压输出
- C4 pad 2: GND -> 地
- C5 pad 1: VCCOUT -> 逻辑板5V_稳压输出
- C5 pad 2: GND -> 地
- C58 pad 1: VCCIN -> 电池保护后母线
- C58 pad 2: GND -> 地
- C59 pad 1: VCCIN -> 电池保护后母线
- C59 pad 2: GND -> 地
- C60 pad 1: VCCIN -> 电池保护后母线
- C60 pad 2: GND -> 地
- C7 pad 1: VCCOUT -> 逻辑板5V_稳压输出
- C8 pad 1: GND -> 降压电源输入
- C8 pad 2: VCCIN -> 地
- C9 pad 1: GND -> 降压电源输入
- C9 pad 2: VCCIN -> 地
- CN1 pad 1: GND -> 地
- CN1 pad 2: VCCIN -> /三串电池输入与电压保护/电池正极
- D1 pad 1: /VM -> 电池保护后母线
- D1 pad 2: GND -> 地
- J1 pad 1: /LAIN1 -> 左电机_原始正转脉宽
- J1 pad 2: /LAIN2 -> 左电机_原始反转脉宽
- J1 pad 3: /LBIN1 -> 电机解锁脉冲
- J1 pad 4: /LBIN2 -> 电机运行许可
- J1 pad 5: GND -> 地
- J1 pad 6: /3.3V -> 逻辑板3.3V_输入
- J1 pad 7: /LF_ENA -> 左编码器_A_逻辑板输入
- J1 pad 8: /LF_ENB -> 左编码器_B_逻辑板输入
- J2 pad 1: /RF_ENB -> 右编码器_B_逻辑板输入
- J2 pad 2: /RF_ENA -> 右编码器_A_逻辑板输入
- J2 pad 3: /3.3V -> 逻辑板3.3V_输入
- J2 pad 4: GND -> 地
- J2 pad 5: /RAIN1 -> 右电机_原始正转脉宽
- J2 pad 6: /RAIN2 -> 右电机_原始反转脉宽
- J2 pad 7: /RBIN1 -> 外部故障_低有效
- J2 pad 8: /RBIN2 -> 电机已解锁
- J3 pad 1: /LAOUT2 -> Net-(J3-Pin_1)
- J3 pad 2: /3.3V -> 本板3.3V
- J3 pad 3: /LF_ENA -> 左编码器_A
- J3 pad 4: /LF_ENB -> 左编码器_B
- J3 pad 5: GND -> 地
- J3 pad 6: /LAOUT1 -> Net-(J3-Pin_6)
- J4 pad 1: /RAOUT2 -> Net-(J4-Pin_1)
- J4 pad 2: /3.3V -> 本板3.3V
- J4 pad 3: /RF_ENA -> 右编码器_A
- J4 pad 4: /RF_ENB -> 右编码器_B
- J4 pad 5: GND -> 地
- J4 pad 6: /RAOUT1 -> Net-(J4-Pin_6)
- L1 pad 1: VCCOUT -> Net-(U5-SW)
- L1 pad 2: Net-(U5-SW) -> 逻辑板5V_稳压输出
- L2 pad 1: VCCOUT1 -> Net-(U1-SW)
- L2 pad 2: Net-(U1-SW) -> 计算板5V_稳压输出
- R1 pad 1: Net-(C6-Pad1) -> Net-(U5-BST)
- R1 pad 2: Net-(U5-BST) -> Net-(C6-Pad1)
- R11 pad 1: VCCOUT1 -> 计算板5V_稳压输出
- R12 pad 2: GND -> 地
- R2 pad 1: VCCOUT -> 逻辑板5V_稳压输出
- R3 pad 2: GND -> 地
- R6 pad 1: Net-(C14-Pad1) -> Net-(U1-BST)
- R6 pad 2: Net-(U1-BST) -> Net-(C14-Pad1)
- U1 pad 1: GND -> 地
- U1 pad 2: VCCIN -> 降压电源输入
- U1 pad 4: GND -> 地
- U1 pad 6: Net-(U1-EN) -> 降压使能
- U5 pad 1: GND -> 地
- U5 pad 2: VCCIN -> 降压电源输入
- U5 pad 4: GND -> 地
- U5 pad 6: Net-(U5-EN) -> 降压使能
Routing:
- net VCCIN: track 153.6 -> 0.00 mm, vias 4 -> 0
- net /3.3V: track 135.2 -> 0.00 mm
- net /VM: track 126.4 -> 0.00 mm, vias 1 -> 0
- net /RAOUT1: track 86.6 -> 0.00 mm
- net VCCOUT1: track 69.6 -> 0.00 mm
- net /RAOUT2: track 61.2 -> 0.00 mm
- net /RBIN1: track 51.2 -> 0.00 mm, vias 3 -> 0
- net /RBIN2: track 48.0 -> 0.00 mm, vias 5 -> 0
- net /LAOUT2: track 47.6 -> 0.00 mm
- net /LAOUT1: track 44.1 -> 0.00 mm
- net /LBIN1: track 43.1 -> 0.00 mm
- net /LBIN2: track 41.7 -> 0.00 mm
- net VCCOUT: track 39.5 -> 0.00 mm
- net /LAIN1: track 34.9 -> 0.00 mm, vias 2 -> 0
- net /LAIN2: track 34.3 -> 0.00 mm, vias 4 -> 0
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- removed copper zone on F.Cu, net /VM
- removed copper zone on B.Cu, net GND
- removed copper zone on F.Cu, net GND
- removed copper zone on F.Cu, net Net-(U1-SW)
- removed copper zone on F.Cu, net Net-(U5-SW)
- removed copper zone on F.Cu, net VCCIN
- removed copper zone on F.Cu, net VCCOUT
- removed copper zone on F.Cu, net VCCOUT1
Other:
- board outline removed

Commit message: 10.3
Parts:
- moved R67 174.8 mm to (78.0, 51.7)
- moved R68 174.8 mm to (78.0, 49.2)
- moved USB2 174.8 mm to (69.5, 43.5)
- moved U8 174.4 mm to (70.0, 50.5), turned to -90 degrees
- moved C1 169.6 mm to (64.5, 62.8)
- moved C11 169.6 mm to (73.4, 62.8)
- moved C2 169.6 mm to (64.5, 65.8)
- moved C3 169.6 mm to (64.5, 68.8)
- moved C4 169.6 mm to (64.5, 71.8)
- moved L1 169.6 mm to (67.3, 77.4)
- moved R2 169.6 mm to (78.3, 74.6)
- moved R3 169.6 mm to (78.3, 77.1)
- moved C5 169.6 mm to (69.0, 62.8)
- moved C6 169.6 mm to (74.2, 74.6)
- moved C7 169.6 mm to (74.2, 77.1)
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Connections:
- net /三串电池输入与电压保护/电池正极 renamed BAT_POS
- net 上电复位完成 renamed POR_OK
- net 传感器3.3V renamed +3V3_SENS
- net 供电口1_总线电源 renamed USB1_VBUS
- net 供电口1_故障脉冲_低有效 renamed USB1_FAULT_PULSE_N
- net 供电口2_总线电源 renamed USB2_VBUS
- net 供电口2_故障脉冲_低有效 renamed USB2_FAULT_PULSE_N
- net 右电机_动力电源 renamed VM_R
- net 右电机_原始反转脉宽 renamed R_PWM_REV_RAW
- net 右电机_原始正转脉宽 renamed R_PWM_FWD_RAW
- net 右电机_母线电流采样 renamed VM_R_IMON
- net 右电机_限流参考 renamed VREF_R
- net 右编码器_A renamed ENC_R_A
- net 右编码器_A_逻辑板输入 renamed ENC_R_A_FPGA
- net 右编码器_B renamed ENC_R_B
- net 右编码器_B_逻辑板输入 renamed ENC_R_B_FPGA
- net 地 renamed GND
- net 基准电压_2.495V renamed VREF_2V495
- net 外部故障_低有效 renamed EXT_KILL_N
- net 左电机_动力电源 renamed VM_L
- net 左电机_原始反转脉宽 renamed L_PWM_REV_RAW
- net 左电机_原始正转脉宽 renamed L_PWM_FWD_RAW
- net 左电机_母线电流采样 renamed VM_L_IMON
- net 左电机_限流参考 renamed VREF_L
- net 左编码器_A renamed ENC_L_A
- net 左编码器_A_逻辑板输入 renamed ENC_L_A_FPGA
- net 左编码器_B renamed ENC_L_B
- net 左编码器_B_逻辑板输入 renamed ENC_L_B_FPGA
- net 急停回路闭合 renamed ESTOP_OK
- net 本板3.3V renamed +3V3
- net 板载3.3V_保护输出 renamed +3V3_ONBOARD
- net 板载3.3V_电压正常 renamed 3V3_ONBOARD_OK
- net 板载3.3V_稳压输出 renamed +3V3_RAW
- net 电机供电正常 renamed MOTOR_POWER_OK
- net 电机已解锁 renamed MOTOR_ARMED
- net 电机总开关输出 renamed VM_SWITCHED
- net 电机解锁脉冲 renamed MOTOR_ARM
- net 电机运行许可 renamed MOTOR_PERMIT
- net 电池保护后母线 renamed VBAT_SYS
- net 电池欠压告警_低有效 renamed BAT_WARN_N
- net 电池电压采样 renamed BAT_ADC
- net 计算板5V_保护输出 renamed +5V_AI_PROT
- net 计算板5V_电压正常 renamed +5V_AI_OK
- net 计算板5V_稳压输出 renamed +5V_AI
- net 过流基准_1.217V renamed CURRENT_REF_1V217
- net 逻辑板3.3V_输入 renamed 3V3_FPGA_IN
- net 逻辑板5V_保护输出 renamed +5V_FPGA_PROT
- net 逻辑板5V_电压正常 renamed +5V_FPGA_OK
- net 逻辑板5V_稳压输出 renamed +5V_FPGA
- net 降压使能 renamed BUCK_ENABLE
- net 降压电源输入 renamed VLOGIC_IN
Routing:
- net VBAT_SYS: track 0.00 -> 32.2 mm
- net Net-(D3-A): track 0.00 -> 15.2 mm
- net Net-(D2-A): track 0.00 -> 6.83 mm
- net VLOGIC_IN: track 0.00 -> 6.60 mm
- net Net-(Q4-B): track 0.00 -> 2.06 mm
- added copper zone on F.Cu, net BAT_POS
- added copper zone on F.Cu, net Net-(Q1-D)

Commit message: 10.4
Parts:
- moved U11 78.6 mm to (123.9, 185.1)
- moved C101 51.8 mm to (58.0, 65.8), turned to 90 degrees
- moved R54 49.1 mm to (47.6, 58.2)
- moved Q3 46.6 mm to (49.2, 63.3), turned to -90 degrees
- moved C103 43.6 mm to (82.0, 70.9)
- moved Q4 43.1 mm to (45.9, 61.3), turned to -90 degrees
- moved R59 41.5 mm to (61.6, 70.8)
- moved U21 40.6 mm to (73.8, 79.5), turned to 0 degrees
- moved C102 40.2 mm to (68.4, 70.9)
- moved R60 40.0 mm to (73.2, 75.3)
- moved R53 36.8 mm to (44.4, 65.8), turned to 90 degrees
- moved R63 35.5 mm to (83.8, 76.9)
- moved R52 34.9 mm to (70.2, 79.5), turned to 0 degrees
- moved D3 34.8 mm to (46.4, 65.8), turned to 90 degrees
- moved R62 34.7 mm to (83.8, 75.3), turned to 180 degrees
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Routing:
- net VBAT_SYS: track 32.2 -> 93.8 mm, vias 0 -> 2
- net VREF_2V495: track 0.00 -> 39.3 mm
- net BUCK_ENABLE: track 0.00 -> 29.6 mm, vias 0 -> 2
- net +5V_FPGA: track 0.00 -> 29.1 mm, vias 0 -> 2
- net VLOGIC_IN: track 6.60 -> 24.8 mm
- net Net-(D3-A): track 15.2 -> 7.72 mm
- net MOTOR_POWER_OK: track 0.00 -> 7.44 mm
- net Net-(U5-SW): track 0.00 -> 7.16 mm
- net Net-(U5-FB): track 0.00 -> 5.76 mm
- net Net-(U22B--): track 0.00 -> 3.64 mm
- net Net-(U23B--): track 0.00 -> 3.61 mm
- net Net-(U23A-+): track 0.00 -> 3.48 mm
- net Net-(U5-VCC): track 0.00 -> 2.44 mm
- net Net-(C6-Pad1): track 0.00 -> 1.61 mm
- net Net-(U5-BST): track 0.00 -> 1.45 mm
- added copper zone on F.Cu, net Net-(U22A-+)

Commit message: 10.8
Parts:
- moved R110 182.3 mm to (60.6, 43.5), turned to 180 degrees
- moved R109 178.3 mm to (64.0, 43.5), turned to 180 degrees
- moved R111 177.3 mm to (65.9, 46.0), turned to 180 degrees
- moved R113 176.5 mm to (66.9, 50.7)
- moved R112 175.8 mm to (69.2, 44.5), turned to -90 degrees
- moved D8 173.2 mm to (71.2, 43.6), turned to -90 degrees
- moved C140 173.1 mm to (63.6, 54.0), turned to -90 degrees
- moved U28 170.5 mm to (61.7, 48.5), turned to -90 degrees
- moved Q11 165.0 mm to (69.2, 48.0), turned to -90 degrees
- moved Q10 153.7 mm to (75.2, 47.8), turned to -90 degrees
- moved R106 152.6 mm to (96.8, 62.5), turned to -90 degrees
- moved U27 149.9 mm to (99.5, 67.0)
- moved D7 146.2 mm to (95.2, 57.3)
- moved R104 143.6 mm to (94.8, 65.0), turned to -90 degrees
- moved R105 143.6 mm to (94.8, 68.0), turned to -90 degrees
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Routing:
- net +5V_AI: track 0.00 -> 14.8 mm
- net USB2_VBUS: track 0.00 -> 12.3 mm
- net USB1_VBUS: track 0.00 -> 11.8 mm
- net +5V_FPGA: track 29.1 -> 39.7 mm
- net Net-(D7-A): track 0.00 -> 8.31 mm
- net Net-(D8-A): track 0.00 -> 7.81 mm
- net +5V_FPGA_OK: track 0.00 -> 7.12 mm
- net Net-(Q9-B): track 0.00 -> 6.98 mm
- net +5V_AI_OK: track 0.00 -> 6.69 mm
- net Net-(U8-CC2): track 0.00 -> 6.32 mm, vias 0 -> 2
- net Net-(U7-CC2): track 0.00 -> 5.85 mm, vias 0 -> 2
- net +5V_FPGA_PROT: track 0.00 -> 5.83 mm
- net Net-(Q11-B): track 0.00 -> 5.65 mm
- net Net-(U8-CC1): track 0.00 -> 5.55 mm
- net Net-(U7-CC1): track 0.00 -> 5.08 mm
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- added copper zone on F.Cu, net +5V_AI
- added copper zone on F.Cu, net +5V_FPGA
- added copper zone on F.Cu, net +5V_FPGA_PROT
