File: pcb/power/kicad/ProPrj_power_2026-10-02.kicad_pcb (KiCad board)
At the start: 2 copper layers, 211 parts, among them CN1 XT60PW-M / 三串电池, J1 左轮控制, J10 惯性传感器电源, J11 测距传感器1电源, J12 测距传感器2电源, J13 测距传感器3电源, J14 3.3V辅助输出, J15 急停常闭回路, J16 左回生泄放 / 外接3.3Ω, J17 右回生泄放 / 外接3.3Ω, J18 电源监测 / 外部模数转换, J2 右轮控制, J3 MG513电机 / 核对线序, J4 MG513电机 / 核对线序, J9 可选逻辑板3.3V输入, Q1 IRF4905, Q10 AO4409, Q11 MMBT3904, Q12 AO3401A, Q13 MMBT3904, Q2 IRF4905, Q3 IRF4905, Q4 MMBT3904, Q5 MMBT3904, Q6 IRLZ44N, Q7 IRLZ44N, Q8 AO4409, Q9 MMBT3904, U1 MP2236GJ-Z, U10 74HC08D, U11 74HC08D, U12 74HC74D, U13 MCP100-300DI/TO, U2 AT8236双路模块, U21 TL431BIDBZR, U22 LM393BIDR, U23 LM393BIDR, U24 LM393BIDR, U25 INA180A1IDBVR, U26 INA180A1IDBVR, U27 LM393BIDR, U28 LM393BIDR, U29 LM393BIDR, U3 AP63203WU-7, U30 LM393BIDR, U4 AT8236双路模块, U5 MP2236GJ-Z, U7 HUSB305-02, U8 HUSB305-02

Commit message: 10.8
Parts:
- moved C106 20.0 mm to (84.2, 50.5)
- moved C107 20.0 mm to (72.8, 47.5)
- moved R67 20.0 mm to (88.0, 48.7)
- moved R68 20.0 mm to (88.0, 46.2)
- moved U8 20.0 mm to (78.9, 47.7)
- moved USB2 20.0 mm to (79.5, 40.5)
Routing:
- net BUCK_ENABLE: track 29.6 -> 45.0 mm, vias 2 -> 3
Changed lines of the file:
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@@
 	(footprint "Package_TO_SOT_SMD:TSOT-23-8"
 		(layer "F.Cu")
-		(at 93 33.5 90)
+		(at 78.885 47.7125 90)
 		(descr "TSOT, 8 Pin (https://www.jedec.org/sites/default/files/docs/MO-193D.pdf variant BA)")
 		(tags "TSOT TO_SOT_SMD")
@@
 	(footprint "Resistor_SMD:R_0603_1608Metric"
 		(layer "F.Cu")
-		(at 102.11 31.9875 180)
+		(at 87.995 46.2 180)
 		(descr "Resistor SMD 0603 (1608 Metric), square (rectangular) end terminal, IPC-7351 nominal, (Body size source: IPC-SM-782 page 72, https://www.pcb-3d.com/wordpress/wp-content/uploads/ipc-sm-782a_amendment_1_and_2.pdf)")
 		(tags "resistor")
@@
 	(footprint "Capacitor_SMD:C_0805_2012Metric"
 		(layer "F.Cu")
-		(at 86.865 33.2875 180)
+		(at 72.75 47.5 180)
 		(descr "Capacitor SMD 0805 (2012 Metric), square (rectangular) end terminal, IPC-7351 nominal, (Body size source: IPC-SM-782 page 76, https://www.pcb-3d.com/wordpress/wp-content/uploads/ipc-sm-782a_amendment_1_and_2.pdf, https://docs.google.com/spreadsheets/d/1BsfQQcO9C6DZCsRaXUlFlo91Tg2WpOkGARC1WS5S8t0/edit?usp=sharing)")
 		(tags "capacitor")
@@
 	(footprint "Connector_USB:USB_C_Receptacle_GCT_USB4125-xx-x_6P_TopMnt_Horizontal"
 		(layer "F.Cu")
-		(at 93.615 26.2875 180)
+		(at 79.5 40.5 180)
 		(descr "USB Type C Receptacle, GCT, power-only, 6P, top mounted, horizontal, 3A, 1mm stake: https://gct.co/files/drawings/usb4125.pdf")
 		(tags "USB C Type-C receptacle power-only charging-only 6P 6C right angled")
@@
 	(footprint "Capacitor_SMD:C_0805_2012Metric"
 		(layer "F.Cu")
-		(at 98.365 36.2875 180)
+		(at 84.25 50.5 180)
 		(descr "Capacitor SMD 0805 (2012 Metric), square (rectangular) end terminal, IPC-7351 nominal, (Body size source: IPC-SM-782 page 76, https://www.pcb-3d.com/wordpress/wp-content/uploads/ipc-sm-782a_amendment_1_and_2.pdf, https://docs.google.com/spreadsheets/d/1BsfQQcO9C6DZCsRaXUlFlo91Tg2WpOkGARC1WS5S8t0/edit?usp=sharing)")
 		(tags "capacitor")
@@
 	(footprint "Resistor_SMD:R_0603_1608Metric"
 		(layer "F.Cu")
-		(at 102.11 34.4975 180)
+		(at 87.995 48.71 180)
 		(descr "Resistor SMD 0603 (1608 Metric), square (rectangular) end terminal, IPC-7351 nominal, (Body size source: IPC-SM-782 page 72, https://www.pcb-3d.com/wordpress/wp-content/uploads/ipc-sm-782a_amendment_1_and_2.pdf)")
 		(tags "resistor")
@@
 	)
 	(segment
+		(start 68.758435 57.741565)
+		(end 67.5 59)
+		(width 0.4)
+		(layer "F.Cu")
+		(net "BUCK_ENABLE")
+	)
+	(segment
+		(start 71.25 57.370926)
+		(end 70.879361 57.741565)
+		(width 0.4)
+		(layer "F.Cu")
+		(net "BUCK_ENABLE")
+	)
+	(segment
+		(start 70.879361 57.741565)
+		(end 68.758435 57.741565)
+		(width 0.4)
+		(layer "F.Cu")
+		(net "BUCK_ENABLE")
+	)
+	(segment
 		(start 64.235 72.7475)
 		(end 65.505 74.0175)
@@
 	)
 	(segment
+		(start 67.5 59)
+		(end 62.5 59)
+		(width 0.4)
+		(layer "F.Cu")
+		(net "BUCK_ENABLE")
+	)
+	(segment
 		(start 62.415 72.7475)
 		(end 64.235 72.7475)
@@
 	)
 	(segment
+		(start 71.25 56.6125)
+		(end 71.25 57.370926)
+		(width 0.4)
+		(layer "F.Cu")
+		(net "BUCK_ENABLE")
+	)
+	(segment
 		(start 51 58.25)
 		(end 48.465 58.25)
@@
 	)
 	(via
+		(at 62.5 59)
+		(size 0.5)
+		(drill 0.3)
+		(layers "F.Cu" "B.Cu")
+		(net "BUCK_ENABLE")
+	)
+	(via
 		(at 51 58.25)
 		(size 0.6)
@@
 	)
 	(segment
+		(start 62.5 59)
+		(end 60 61.5)
+		(width 0.4)
+		(layer "B.Cu")
+		(net "BUCK_ENABLE")
+	)
+	(segment
 		(start 62.415 69.5)
 		(end 62.415 65.665)
@@
 		(layer "B.Cu")
 		(net "BUCK_ENABLE")
+	)
+	(segment
+		(start 60 61.5)
+		(end 60 63.25)
+		(width 0.4)
+		(layer "B.Cu")
+		(net "BUCK_ENABLE")
