File: pcb/power/kicad/ProPrj_power_2026-10-02.kicad_pcb (KiCad board)
At the start: 2 copper layers, 211 parts, among them CN1 XT60PW-M / 三串电池, J1 左轮控制, J10 惯性传感器电源, J11 测距传感器1电源, J12 测距传感器2电源, J13 测距传感器3电源, J14 3.3V辅助输出, J15 急停常闭回路, J16 左回生泄放 / 外接3.3Ω, J17 右回生泄放 / 外接3.3Ω, J18 电源监测 / 外部模数转换, J2 右轮控制, J3 MG513电机 / 核对线序, J4 MG513电机 / 核对线序, J9 可选逻辑板3.3V输入, Q1 IRF4905, Q10 AO4409, Q11 MMBT3904, Q12 AO3401A, Q13 MMBT3904, Q2 IRF4905, Q3 IRF4905, Q4 MMBT3904, Q5 MMBT3904, Q6 IRLZ44N, Q7 IRLZ44N, Q8 AO4409, Q9 MMBT3904, U1 MP2236GJ-Z, U10 74HC08D, U11 74HC08D, U12 74HC74D, U13 MCP100-300DI/TO, U2 AT8236双路模块, U21 TL431BIDBZR, U22 LM393BIDR, U23 LM393BIDR, U24 LM393BIDR, U25 INA180A1IDBVR, U26 INA180A1IDBVR, U27 LM393BIDR, U28 LM393BIDR, U29 LM393BIDR, U3 AP63203WU-7, U30 LM393BIDR, U4 AT8236双路模块, U5 MP2236GJ-Z, U7 HUSB305-02, U8 HUSB305-02

Commit message: Update ProPrj_power_2026-10-02.kicad_pcb
Parts:
- moved R104 6.86 mm to (88.0, 66.2)
- moved C139 6.86 mm to (98.5, 66.3)
- moved Q9 6.86 mm to (93.3, 60.5)
- moved R105 6.86 mm to (88.0, 69.2)
- moved R107 6.86 mm to (89.3, 60.5)
- moved R108 6.86 mm to (95.0, 62.9)
- moved U27 6.86 mm to (92.8, 68.2)
- moved D7 6.86 mm to (88.4, 58.5)
- moved R106 6.86 mm to (90.1, 63.7)
- moved C104 6.86 mm to (94.0, 50.5)
- moved C105 6.86 mm to (94.0, 48.5)
- moved Q8 6.86 mm to (92.7, 54.5)
- moved R65 6.86 mm to (97.8, 53.2)
- moved R66 6.86 mm to (96.5, 46.0)
- moved U7 6.86 mm to (97.5, 49.5)
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
Commit message: 10.12
Parts:
- moved Q6 226.4 mm to (30.5, 70.0), turned to 90 degrees
- moved D4 224.6 mm to (36.2, 94.0)
- moved Q5 219.6 mm to (41.0, 94.0), turned to -90 degrees
- moved R74 214.9 mm to (38.2, 89.8), turned to 90 degrees
- moved TP1 211.9 mm to (49.0, 97.5)
- moved R123 210.6 mm to (44.8, 53.0), turned to -90 degrees
- moved J16 210.3 mm to (30.9, 82.5), turned to -90 degrees
- moved R122 209.6 mm to (44.8, 56.8), turned to -90 degrees
- moved R75 207.0 mm to (45.2, 97.0), turned to 180 degrees
- moved D5 206.5 mm to (55.8, 94.2), turned to 90 degrees
- moved Q2 204.3 mm to (46.0, 94.0)
- moved R78 201.0 mm to (57.0, 86.5), turned to 180 degrees
- moved U30 191.7 mm to (50.0, 53.0)
- moved C142 190.3 mm to (56.0, 51.0)
- moved R76 189.4 mm to (67.2, 87.2)
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Routing:
- net +3V3: track 0.00 -> 493.8 mm, vias 0 -> 5
- net VBAT_SYS: track 98.0 -> 332.3 mm, vias 2 -> 8
- net MOTOR_POWER_OK: track 7.44 -> 226.2 mm, vias 0 -> 10
- net +3V3_SENS: track 0.00 -> 210.3 mm, vias 0 -> 9
- net MOTOR_ARMED: track 0.00 -> 194.2 mm, vias 0 -> 9
- net 3V3_FPGA_IN: track 0.00 -> 186.1 mm, vias 0 -> 7
- net ESTOP_OK: track 0.00 -> 184.6 mm, vias 0 -> 7
- net VM_L_IMON: track 0.00 -> 143.6 mm, vias 0 -> 10
- net VM_R_IMON: track 0.00 -> 134.2 mm, vias 0 -> 8
- net VREF_2V495: track 39.3 -> 171.7 mm, vias 0 -> 10
- net +5V_AI: track 14.8 -> 141.9 mm, vias 0 -> 8
- net POR_OK: track 0.00 -> 126.6 mm, vias 0 -> 9
- net GND: track 0.00 -> 108.6 mm, vias 0 -> 115
- net Net-(U4-AIN2): track 0.00 -> 102.0 mm, vias 0 -> 6
- net BUCK_ENABLE: track 45.0 -> 141.8 mm, vias 3 -> 9
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- added copper zone on F.Cu, net +5V_AI_PROT
- added copper zone on B.Cu, net BAT_POS
- added copper zone on B.Cu, net GND
- added copper zone on F.Cu, net GND
- added copper zone on B.Cu, net Net-(Q1-D)
- added copper zone on B.Cu, net VM_L
- added copper zone on F.Cu, net VM_L
- added copper zone on B.Cu, net VM_R
- added copper zone on F.Cu, net VM_R
- added copper zone on B.Cu, net VM_SWITCHED
- added copper zone on F.Cu, net VM_SWITCHED
Other:
- board outline added: 96 x 97 mm
- board text added: "双层电源板"

Commit message: 10.16
Routing:
- net VM_R: track 61.2 -> 62.9 mm
- removed copper zone on B.Cu, net GND
- removed copper zone on F.Cu, net GND
